File: hw/panel/panel.kicad_pcb (KiCad board)
At the start: 4 copper layers, 158 x 89 mm, 296 parts, among them J1 Input, J1 USB_OTG, J2 BATT, J2 Output, J201 Modem, J202 SIM_Card, J203 Motor, J204 Micro_SD_Card, J205 Prog, J206 Expansion, J207 Camera, J3 +5V, J301 iMX8, J305 Micro_SD_Card, J4 SJ-3571N, J401 Touch, J402 Display, J5 SPEAKER, SW1 RESET, SW2 WAKE, SW201 BOOT, SW202 PERST, U1 BQ25895, U1 SN65LVDS822, U10 74HC595, U11 ICS-43434, U12 MAX98357A, U13 MAX98357A, U14 SN74LVC1G04DCK, U15 SN74LVC1G3157DCK, U16 SN74LVC2G07DCK, U2 SN74LVC00ARGY, U2 TPS62293, U201 ESP32-WROOM, U202 SN74CBTLV3125RGY, U203 TXB0104RGY, U204 TXB0104RGY, U205 DRV2605LDGS, U206 LSM9DS1, U207 FT230XQ, U208 TMUX154ERSW, U3 TPS630250, U4 FE310-G002, U401 FAN5333BSX, U402 SN74LVC3G06DCU, U403 BT817Q, U404 IS25LP128-JKLE, U405 DS90C185, U406 TS3DV520ERUA, U407 TXS0104ERGY, U408 TXS0104ERGY, U409 SN74LVC2G06DCK, U5 IS25LP128-JKLE, U6 TMUX1574RSV, U7 74HC00, U8 74HC00, U9 74HC595, X1 SiT1533, Y1 16MHz, Y401 12MHz

Commit message: temp commit for merge
Parts:
- removed the C1 at (189.5, 86.6)
- removed the C1 at (58.2, 111.5)
- removed the C11 at (186.7, 91.3)
- removed the C11 at (92.0, 117.5)
- removed C439, C440: 0.1uF, Capacitor_SMD:C_0603_1608Metric
- removed the J1 at (194.6, 95.1)
- removed the J1 at (68.3, 123.4)
- removed the J2 at (199.6, 67.9)
- removed the J2 at (57.5, 122.0)
- removed the J3 at (61.9, 122.0)
- removed J305: Micro_SD_Card, footprints:microSD
- removed the R2 at (69.1, 112.6)
- removed the R3 at (67.4, 117.9)
- removed the R4 at (67.6, 111.1)
- removed R414, R415: R, Resistor_SMD:R_0603_1608Metric
- removed the R5 at (90.5, 124.3)
- removed the R6 at (88.2, 125.0)
- removed the REF** at (183.5, 114.5)
- removed the REF** at (183.5, 82.0)
- removed the REF** at (98.0, 127.5)
- removed the REF** at (140.0, 127.5)
- removed the REF** at (200.0, 127.5)
- removed the REF** at (200.0, 101.5)
- removed the REF** at (200.0, 61.5)
- removed the U2 at (205.3, 81.8)
- removed the U2 at (59.6, 100.8)
- added C1: 47nF, Capacitor_SMD:C_0603_1608Metric, F.Cu at (58.3, 120.0)
- added C1: 0.1uF, Capacitor_SMD:C_0603_1608Metric, B.Cu at (209.4, 81.0)
- added C11: 47uF, Capacitor_SMD:C_0805_2012Metric, F.Cu at (106.8, 122.3)
- added C11: 10uF, Capacitor_SMD:C_0603_1608Metric, F.Cu at (212.1, 69.7)
- added C13: 0.1uF, Capacitor_SMD:C_0603_1608Metric, F.Cu at (216.1, 64.2)
- added C228: 22uF, Capacitor_SMD:C_0805_2012Metric, F.Cu at (141.3, 114.7)
- added C320: 22uF, Capacitor_SMD:C_0805_2012Metric, B.Cu at (66.3, 83.0)
- added J1: USB_OTG, footprints:GCT_MicroUSB-USB3080, F.Cu at (68.9, 126.9)
- added J1: Input, Connector_Molex:Molex_SlimStack_55560-0301_2x15_P0.50mm_Vertical, F.Cu at (206.1, 72.4)
- added J1: In, Connector_Molex:Molex_SlimStack_55560-0161_2x08_P0.50mm_Vertical, B.Cu at (199.0, 112.3)
- added J2: BATT, Connector_PinHeader_2.54mm:PinHeader_1x02_P2.54mm_Vertical, F.Cu at (58.0, 111.2)
- added J2: Display, Connector_FFC-FPC:Hirose_FH12-45S-0.5SH_1x45-1MP_P0.50mm_Horizontal, B.Cu at (199.3, 96.7)
- added J2: Out, Connector_PinHeader_2.54mm:PinHeader_2x08_P2.54mm_Vertical, F.Cu at (191.6, 128.7)
- added J3: +5V, Connector_PinHeader_2.54mm:PinHeader_1x02_P2.54mm_Vertical, F.Cu at (60.4, 129.2)
- added J3: Touch, Connector_FFC-FPC:Hirose_FH12-8S-0.5SH_1x08-1MP_P0.50mm_Horizontal, B.Cu at (217.6, 66.0)
- added J302: Micro_SD_Card_Det, footprints:Molex_MicroSD-5027740891, B.Cu at (70.8, 63.3)
- added J303: Spacer, footprints:Spacer, F.Cu at (70.4, 111.9)
- added J4: Spacer, footprints:Spacer, F.Cu at (215.8, 103.1)
- added J403: Spacer, footprints:Spacer, B.Cu at (172.9, 91.0)
- added J5: Spacer, footprints:Spacer, F.Cu at (205.2, 103.1)
- added JP302: USB_ID, Jumper:SolderJumper-2_P1.3mm_Open_RoundedPad1.0x1.5mm, B.Cu at (58.6, 82.2)
- added R2: 10K, Resistor_SMD:R_0603_1608Metric, F.Cu at (69.2, 121.0)
- added R2: DNP, Resistor_SMD:R_0603_1608Metric, F.Cu at (219.5, 76.1)
- added R23: 100K, Resistor_SMD:R_0603_1608Metric, F.Cu at (96.0, 85.7)
- added R24: 100K, Resistor_SMD:R_0603_1608Metric, F.Cu at (94.5, 85.7)
- added R25: 100K, Resistor_SMD:R_0603_1608Metric, F.Cu at (97.5, 85.7)
- added R3: 2.2K, Resistor_SMD:R_0603_1608Metric, B.Cu at (64.3, 126.3)
- added R3: DNP, Resistor_SMD:R_0603_1608Metric, F.Cu at (218.0, 76.1)
- added R301: 100K, Resistor_SMD:R_0603_1608Metric, B.Cu at (70.8, 81.3)
- added R31: 100K, Resistor_SMD:R_0603_1608Metric, F.Cu at (150.2, 93.3)
- added R4: 10K, Resistor_SMD:R_0603_1608Metric, F.Cu at (67.7, 119.5)
- added R4: DNP, Resistor_SMD:R_0603_1608Metric, F.Cu at (216.5, 76.1)
- added R5: 560K, Resistor_SMD:R_0603_1608Metric, F.Cu at (113.7, 123.8)
- added R5: DNP, Resistor_SMD:R_0603_1608Metric, F.Cu at (198.0, 74.8)
- added R6: 180K, Resistor_SMD:R_0603_1608Metric, F.Cu at (114.4, 126.0)
- added R6: DNP, Resistor_SMD:R_0603_1608Metric, F.Cu at (198.0, 73.2)
- added REF**: mouse-bite-3mm-slot, panelization:mouse-bite-3mm-slot, F.Cu at (183.5, 119.9)
- added REF**: mouse-bite-3mm-slot, panelization:mouse-bite-3mm-slot, F.Cu at (183.5, 84.4)
- added REF**: mouse-bite-3mm-slot, panelization:mouse-bite-3mm-slot, F.Cu at (98.0, 132.5)
- added REF**: mouse-bite-3mm-slot, panelization:mouse-bite-3mm-slot, F.Cu at (140.0, 132.5)
- added REF**: mouse-bite-3mm-slot, panelization:mouse-bite-3mm-slot, F.Cu at (203.8, 132.5)
- added REF**: mouse-bite-3mm-slot, panelization:mouse-bite-3mm-slot, F.Cu at (203.8, 107.3)
- added REF**: mouse-bite-3mm-slot, panelization:mouse-bite-3mm-slot, F.Cu at (203.8, 61.5)
- added SW301: iMX8_ALT_BOOT, Button_Switch_SMD:SW_SPST_PTS810, F.Cu at (81.7, 114.2)
- added SW302: iMX8_RST, Button_Switch_SMD:SW_SPST_PTS810, F.Cu at (81.7, 118.0)
- added TP2: PMU_OUT0, TestPoint:TestPoint_Pad_D1.5mm, F.Cu at (127.2, 112.8)
- added U2: TPS62293, footprints:TPS62290, F.Cu at (77.2, 127.2)
- added U2: SN74LVC00ARGY, footprints:Texas_S-PVQFN-N14_ThermalVias, F.Cu at (194.3, 85.8)
- C14: value 10nF -> 22uF; footprint Capacitor_SMD:C_0603_1608Metric -> Capacitor_SMD:C_0805_2012Metric; moved to B.Cu
- C219: value 10nF -> 0.1uF
- C220: value 10nF -> 0.1uF; moved to B.Cu
- C319: moved to B.Cu
- J201: footprint footprints:Socket_mPCIe -> footprints:TE_mPCIe-1775862
- J204: value Micro_SD_Card -> Micro_SD_Card_Det; footprint footprints:microSD -> footprints:Molex_MicroSD-5027740891
- J301: footprint footprints:Socket_SODIMM_DDR3_TE_2013289 -> footprints:TE_SODIMMDDR3-2013289
- J401: value Touch -> Display; footprint Connector_FFC-FPC:Hirose_FH12-8S-0.5SH_1x08-1MP_P0.50mm_Horizontal -> Connector_Molex:Molex_SlimStack_54722-0304_2x15_P0.50mm_Vertical
- J402: value Display -> Spacer; footprint Connector_FFC-FPC:Hirose_FH12-26S-0.5SH_1x26-1MP_P0.50mm_Horizontal -> footprints:Spacer
- JP201: value LEVEL EN -> SIMCom_EN
- JP3: footprint Jumper:SolderJumper-2_P1.3mm_Bridged_RoundedPad1.0x1.5mm -> Jumper:SolderJumper-3_P1.3mm_Bridged12_RoundedPad1.0x1.5mm
- JP301: value ALT_BOOT -> USB_VBUS
- L2: footprint footprints:L_Coilcraft_LPS3015 -> footprints:Coilcraft-LPS3015
- L3: footprint footprints:L_Coilcraft_XAL40 -> footprints:Coilcraft-XAL40
- L401: footprint footprints:L_Murata_LQH66SN -> footprints:Murata-LQH66SN
- SW201: value BOOT -> ESP32_RST
- SW202: value PERST -> MODEM_RST
- U10, U9: footprint footprints:74HC595BQ115 -> footprints:DHVQFN-16_2.5x3.5mm_P0.5mm_EP1.0x2.0mm
- U202, U203, U204: footprint Package_DFN_QFN:Texas_S-PVQFN-N14_ThermalVias -> footprints:Texas_S-PVQFN-N14_ThermalVias
- U407, U408: footprint Package_DFN_QFN:Texas_S-PVQFN-N14_ThermalVias -> footprints:DHVQFN-14_2.5x3.0mm_P0.5mm_EP1.0x1.5mm
- U7, U8: footprint footprints:74HC00BQ115 -> footprints:DHVQFN-14_2.5x3.0mm_P0.5mm_EP1.0x1.5mm
- moved C45 61.8 mm to (142.9, 125.8)
- moved U16 61.8 mm to (146.0, 125.8)
- moved R7 58.1 mm to (145.9, 123.7), turned to 0 degrees
- moved SW1 50.2 mm to (145.0, 129.2)
- moved R10 48.7 mm to (148.6, 129.1)
- moved C14 42.6 mm to (89.5, 80.5)
- moved J205 39.1 mm to (136.1, 126.3)
- moved C7 31.8 mm to (74.9, 127.5)
- moved C8 31.8 mm to (78.0, 125.2)
- moved L2 31.8 mm to (81.2, 126.8)
- moved C12 31.4 mm to (189.7, 96.2), turned to 180 degrees
- moved J402 31.3 mm to (172.9, 80.3), turned to 0 degrees
- moved C220 31.2 mm to (142.2, 69.2), turned to 180 degrees
- moved JP1 27.5 mm to (212.4, 79.3), turned to 270 degrees
- moved C13 26.8 mm to (127.0, 116.2)
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- renumbered C13 to C14, C14 to C15, C228 to C229, C229 to C230, C230 to C231, R23 to R26, R24 to R27, R25 to R28, R26 to R29, R27 to R30, R28 to R32, R29 to R33
Connections:
- net Net-(TP401-Pad1) renamed /disp/BT81X_AUDIO
- net Net-(U4-Pad17) renamed /AON_PMU_OUT_1
- C14 pad 1: WAKE -> +1V8
- J204 pad 2: SPI1.SS3 -> GPIO_0
- J204 pad 9: GND -> Net-(J204-Pad9)
- J206 pad 10: UART0.TXD -> TMUX.I2C0.SCL
- J206 pad 11: SPI1.MOSI -> GND
- J206 pad 13: SPI1.MISO -> UART0.TXD
- J206 pad 14: TMUX.I2C0.SDA -> TMUX.GPIO1
- J206 pad 15: SPI1.SCK -> UART0.RXD
- J206 pad 16: TMUX.I2C0.SCL -> TMUX.GPIO0
- J206 pad 5: TMUX.GPIO0 -> SPI1.MOSI
- J206 pad 7: TMUX.GPIO1 -> SPI1.MISO
- J206 pad 8: UART0.RXD -> TMUX.I2C0.SDA
- J206 pad 9: GND -> SPI1.SCK
- J207 pad 1: GPIO_23 -> TMUX.I2C0.SCL
- J207 pad 3: TMUX.I2C0.SCL -> TMUX.I2C0.SDA
- J207 pad 5: TMUX.I2C0.SDA -> SPI1.SS2
- J207 pad 8: BT81X.GPIO0 -> Net-(J207-Pad8)
- J301 pad 165: Net-(J301-Pad165) -> BT81X.GPIO0
- J301 pad 171: Net-(J301-Pad171) -> /exp/RESET
- J301 pad 174: Net-(J301-Pad174) -> iMX8.USB1.ID
- J301 pad 180: Net-(J301-Pad180) -> iMX8.USB1.VBUS
- J301 pad 61: GND -> /exp/SD2_DET
- J401 pad 1: GND -> +3V3
- J401 pad 3: +VCTP -> +1V8
- J401 pad 4: /disp/CTP_SCL -> /disp/DISP_LVDS_A0N
- J401 pad 5: /disp/CTP_SDA -> /disp/CTP_SCL
- J401 pad 6: /disp/CTP_INT -> /disp/DISP_LVDS_A0P
- J401 pad 7: /disp/CTP_RST -> /disp/CTP_SDA
- J402 pad 1: +3V3 -> GND
- JP3 pad 1: /DISP_EN_IC -> Net-(JP3-Pad1)
- JP3 pad 2: Net-(JP3-Pad2) -> /DISP_DE_INV
- JP301 pad 1: /exp/ALT_BOOT -> +3V3
- JP301 pad 2: +3V3 -> iMX8.USB1.VBUS
- R208 pad 2: SPI1.SS3 -> GPIO_0
- R407 pad 2: SPI1.SS2 -> SPI1.SS3
- R408 pad 2: GPIO_0 -> GPIO_23
- SW2 pad 1: WAKE -> GND
- SW2 pad 2: GND -> WAKE
- U1 pad 38: /DISP_EN_IC -> /DISP_DE_INV
- U4 pad 22: Net-(U4-Pad22) -> /AON_PMU_OUT_0
- U403 pad 11: GPIO_0 -> GPIO_23
- U403 pad 6: SPI1.SS2 -> SPI1.SS3
Routing:
- net /exp/RESET: track 0.00 -> 73.1 mm, vias 0 -> 2
- net /BQ_QON: track 28.3 -> 93.0 mm
- net GND: track 570.8 -> 633.6 mm, vias 598 -> 674
- net +1V8: track 127.8 -> 186.8 mm, vias 23 -> 30
- net /exp/SD2_DET: track 0.00 -> 53.6 mm, vias 0 -> 1
- net /exp/ALT_BOOT: track 22.8 -> 65.4 mm, vias 1 -> 2
- net GPIO_0: track 63.7 -> 30.9 mm, vias 3 -> 2
- net SPI1.SS2: track 58.5 -> 88.5 mm
- net +VCTP: track 46.4 -> 16.5 mm, vias 3 -> 2
- net WAKE: track 143.7 -> 117.8 mm
- net CTP.INT: track 0.00 -> 23.8 mm, vias 0 -> 2
- net GPIO_23: track 79.6 -> 55.9 mm, vias 3 -> 5
- net SPI1.SS3: track 33.5 -> 56.9 mm, vias 4 -> 3
- net CTP.RST: track 0.00 -> 22.6 mm, vias 0 -> 1
- net CTP.SDA: track 0.00 -> 22.0 mm, vias 0 -> 2
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- removed copper zone on F.Cu, net +VCTP
- removed copper zone on B.Cu, net DISP_LED_A
- removed copper zone on B.Cu, net Net-(C6-Pad1)
Other:
- board size 158 x 89 mm -> 166.6 x 94 mm
- net class AUDIO removed
- net class BT81X removed
- net class CTP removed
- net class DISPLAY removed
- net class Default: clearance 0.2 -> 0.1524; trace_width 0.25 -> 0.1524; via_dia 0.6 -> 0.508; via_drill 0.3 -> 0.254
- net class FE310 removed
- net class FE310_L removed
- net class USB removed
- net class USB2DIFF removed
- rule pad_to_mask_clearance: 0.05 -> 0
- rule trace_clearance: 0.2 -> 0.1524
- rule via_min_size: 0.5 -> 0.4

Commit message: HW REV 3.0
Parts:
- removed the C1 at (58.3, 120.0)
- removed the C2 at (63.0, 117.7)
- removed the C42 at (61.4, 126.4)
- removed the C43 at (58.0, 125.8)
- removed C435, C436, C437, C438: 0.1uF, Capacitor_SMD:C_0603_1608Metric
- removed the C44 at (58.0, 123.8)
- removed JP3: DE INVERT, Jumper:SolderJumper-3_P1.3mm_Bridged12_RoundedPad1.0x1.5mm
- removed JP401: CTP_PWR, Jumper:SolderJumper-3_P1.3mm_Open_RoundedPad1.0x1.5mm
- removed the R31 at (150.2, 93.3)
- removed R412, R413: 47K, Resistor_SMD:R_0603_1608Metric
- removed TP1: BQ_INT, TestPoint:TestPoint_Pad_D1.5mm
- removed TP401: AUDIO, TestPoint:TestPoint_Pad_D1.5mm
- removed the U1 at (63.4, 121.5)
- removed the U2 at (77.2, 127.2)
- removed the U2 at (194.3, 85.8)
- removed U408: TXS0104ERGY, footprints:DHVQFN-14_2.5x3.0mm_P0.5mm_EP1.0x1.5mm
- removed U409: SN74LVC2G06DCK, Package_TO_SOT_SMD:Texas_R-PDSO-G6
- added C1: 1uF, Capacitor_SMD:C_0603_1608Metric, F.Cu at (64.0, 125.7)
- added C1: 10uF, Capacitor_SMD:C_0603_1608Metric, F.Cu at (220.4, 116.3)
- added C2: 47nF, Capacitor_SMD:C_0603_1608Metric, F.Cu at (61.7, 120.0)
- added C2: 0.1uF, Capacitor_SMD:C_0603_1608Metric, F.Cu at (217.9, 119.0)
- added C39: 0.1uF, Capacitor_SMD:C_0603_1608Metric, B.Cu at (168.2, 112.0)
- added C40: 0.1uF, Capacitor_SMD:C_0603_1608Metric, B.Cu at (168.2, 115.0)
- added C45: 0.1uF, Capacitor_SMD:C_0603_1608Metric, B.Cu at (180.0, 108.0)
- added C50: 10uF, Capacitor_SMD:C_0603_1608Metric, F.Cu at (67.2, 127.5)
- added C51: 22uF, Capacitor_SMD:C_0805_2012Metric, F.Cu at (59.2, 126.5)
- added C52: 22uF, Capacitor_SMD:C_0805_2012Metric, F.Cu at (57.2, 126.5)
- added C53: 10uF, Capacitor_SMD:C_0603_1608Metric, F.Cu at (62.5, 124.5)
- added C54: 10uF, Capacitor_SMD:C_0603_1608Metric, F.Cu at (61.0, 124.5)
- added C9: 10uF, Capacitor_SMD:C_0603_1608Metric, F.Cu at (80.5, 113.7)
- added D2: LED, LED_SMD:LED_0603_1608Metric, B.Cu at (67.7, 129.3)
- added J6: Ext Audio, Connector_Molex:Molex_SlimStack_54722-0164_2x08_P0.50mm_Vertical, F.Cu at (178.2, 113.7)
- added JP1: AUDIO PWR, Jumper:SolderJumper-3_P1.3mm_Open_RoundedPad1.0x1.5mm, B.Cu at (112.1, 125.0)
- added SW303: iMX8_PWR, Button_Switch_SMD:SW_SPST_PTS810, F.Cu at (79.5, 127.2)
- added U1: BQ25895, Package_DFN_QFN:Texas_S-PWQFN-N24_EP2.7x2.7mm_ThermalVias, F.Cu at (66.8, 121.5)
- added U1: PCA9536DP, Package_SON:WSON-8-1EP_3x3mm_P0.5mm_EP1.6x2.0mm, F.Cu at (220.4, 119.7)
- added U15: MAX14689A, footprints:TDFN-10-1EP_2x2.5mm_P0.4mm_EP1.3x1.4mm_ThermalVias, F.Cu at (169.4, 112.0)
- added U16: MAX14689A, footprints:TDFN-10-1EP_2x2.5mm_P0.4mm_EP1.3x1.4mm_ThermalVias, F.Cu at (169.4, 115.0)
- added U19: 74LVC1G02, footprints:Texas_R-PDSO-G5, F.Cu at (180.0, 108.0)
- added U2: TPS62293, footprints:TPS62290, F.Cu at (79.8, 115.7)
- added U2: 74LVC2G00, Package_SO:VSSOP-8_2.3x2mm_P0.5mm, F.Cu at (211.0, 82.6)
- C3: value 10uF -> 4.7uF
- C4: value 1uF -> 10uF
- C5: value 4.7uF -> 10uF
- D1: value LED -> B5817WS; footprint LED_SMD:LED_0603_1608Metric -> footprints:D_SOD-323; moved to F.Cu
- J1: moved to F.Cu
- J303: value Spacer -> Console; footprint footprints:Spacer -> Connector_FFC-FPC:Hirose_FH12-6S-0.5SH_1x06-1MP_P0.50mm_Horizontal; moved to B.Cu
- L1: footprint Inductor_SMD:L_Vishay_IHLP-1616 -> Inductor_SMD:L_Vishay_IHLP-2525
- R2: value 10K -> 5.23K
- R26: value 2.2K -> 100K
- R27: value 255K -> 210K
- R3: value 2.2K -> 30.1K; moved to F.Cu
- R4: value 10K -> 2.2K; moved to B.Cu
- U18: renamed from U15; value SN74LVC1G3157DCK -> TMUX1119DCK
- U407: value TXS0104ERGY -> TMUX1574RSV; footprint footprints:DHVQFN-14_2.5x3.0mm_P0.5mm_EP1.0x1.5mm -> footprints:UQFN-16_1.8x2.6mm_P0.4mm
- moved C13 47.3 mm to (191.6, 104.7), turned to 0 degrees
- moved J303 47.2 mm to (87.5, 67.9)
- moved J3 45.9 mm to (190.1, 102.8), turned to 0 degrees
- moved J4 44.5 mm to (191.8, 65.7), turned to 90 degrees
- moved J5 37.5 mm to (202.4, 65.7), turned to 90 degrees
- moved C12 36.8 mm to (217.9, 72.6), turned to 0 degrees
- moved R2 35.5 mm to (188.1, 92.7), turned to 270 degrees
- moved C11 33.8 mm to (195.5, 99.2), turned to 270 degrees
- moved R11 33.5 mm to (150.1, 129.1), turned to 270 degrees
- moved R3 32.9 mm to (189.6, 92.7), turned to 270 degrees
- moved R4 30.3 mm to (191.1, 92.7), turned to 270 degrees
- moved JP2 29.3 mm to (213.8, 93.8), turned to 180 degrees
- moved J2 26.2 mm to (208.2, 72.1), turned to 180 degrees
- moved R6 25.1 mm to (209.6, 95.5), turned to 180 degrees
- moved J1 24.4 mm to (201.5, 96.4), turned to 180 degrees
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- renumbered C9 to C10, C10 to C11, C11 to C12, C12 to C13, C13 to C14, C45 to C28, C28 to C29, C29 to C30, C30 to C31, C31 to C32, C32 to C33, C33 to C34, C34 to C35, C35 to C36, C36 to C37, C37 to C38, C38 to C41, C39 to C42, C40 to C43, C41 to C44, C14 to C55, R16 to R15, R15 to R16, R32 to R31, R33 to R32, U9 to U10, U10 to U11, U11 to U12, U12 to U13, U13 to U14, U14 to U17, U16 to U6, U6 to U7, U7 to U8, U8 to U9
Connections:
- net /HP_SWITCH renamed /~HP_DET
- net /PIN10 renamed /GPIO0
- C3 pad 1: +VSYS -> Net-(C3-Pad1)
- C35 pad 1: +VSYS -> VDDA
- C36 pad 1: +VSYS -> VDDA
- C37 pad 1: +VSYS -> VDDA
- C38 pad 1: +VSYS -> VDDA
- C4 pad 1: VBUS -> +VSYS
- C41 pad 2: Net-(C38-Pad2) -> /HP_R
- C42 pad 2: Net-(C39-Pad2) -> /HP_L
- C44 pad 1: +VSYS -> VDDA
- C5 pad 1: Net-(C5-Pad1) -> +VSYS
- C7 pad 1: +VSYS -> Net-(C6-Pad1)
- C8 pad 1: +1V8 -> +VSYS
- D1 pad 1: Net-(D1-Pad1) -> /BQ_PMID
- D1 pad 2: +VSYS -> /BQ_SW
- J1 pad 1: /PIN1 -> +3V3
- J1 pad 12: GND -> /I2C_SDA
- J1 pad 13: /PIN13 -> /UART_TX
- J1 pad 14: /PIN14 -> /I2C_SCL
- J1 pad 15: /PIN15 -> /UART_RX
- J1 pad 16: /PIN16 -> GND
- J1 pad 2: /PIN2 -> VDD
- J1 pad 3: GND -> +3V3
- J1 pad 4: /PIN4 -> VDD
- J1 pad 5: /PIN5 -> /SPI_MOSI
- J1 pad 7: /PIN7 -> /SPI_MISO
- J1 pad 8: /PIN8 -> /SPI_CS
- J1 pad 9: /PIN9 -> /SPI_SCK
- J2 pad 1: /PIN1 -> /SPI_CS
- J2 pad 11: GND -> +3V3
- J2 pad 12: GND -> VDD
- J2 pad 13: /PIN13 -> /I2C_SDA
- J2 pad 14: /PIN14 -> /UART_TX
- J2 pad 15: /PIN15 -> /I2C_SCL
- J2 pad 16: /PIN16 -> /UART_RX
- J2 pad 2: /PIN2 -> /PCA_IO3
- J2 pad 3: GND -> /SPI_MOSI
- J2 pad 4: /PIN4 -> /PCA_IO2
- J2 pad 5: /PIN5 -> /SPI_MISO
- J2 pad 6: GND -> /PCA_IO1
- J2 pad 7: /PIN7 -> /SPI_SCK
- J2 pad 8: /PIN8 -> /PCA_IO0
- J2 pad 9: /PIN9 -> GND
- J206 pad 10: TMUX.I2C0.SCL -> Net-(J206-Pad10)
- J206 pad 12: GND -> TMUX.I2C0.SDA
- J206 pad 14: TMUX.GPIO1 -> TMUX.I2C0.SCL
- J206 pad 16: TMUX.GPIO0 -> GND
- J206 pad 2: +VSYS -> VDDA
- J206 pad 3: GND -> +3V3
- J206 pad 4: +VSYS -> VDDA
- J206 pad 8: TMUX.I2C0.SDA -> Net-(J206-Pad8)
- J207 pad 1: TMUX.I2C0.SCL -> +3V3
- J207 pad 10: GND -> BT81X.GPIO0
- J207 pad 11: +VSYS -> GND
- J207 pad 12: GND -> TMUX.I2C0.SDA
- J207 pad 13: +VSYS -> Net-(J207-Pad13)
- J207 pad 14: GND -> TMUX.I2C0.SCL
- J207 pad 15: GND -> Net-(J207-Pad15)
- J207 pad 16: +3V3 -> GND
- J207 pad 2: SPI1.SCK -> +VSYS
- J207 pad 3: TMUX.I2C0.SDA -> +3V3
- J207 pad 4: SPI1.MISO -> +VSYS
- J207 pad 5: SPI1.SS2 -> SPI1.MOSI
- J207 pad 6: SPI1.MOSI -> GND
- J207 pad 7: GND -> SPI1.MISO
- J207 pad 8: Net-(J207-Pad8) -> SPI1.SS2
- J207 pad 9: GND -> SPI1.SCK
- J301 pad 111: Net-(J301-Pad111) -> /exp/UART3_TX
- J301 pad 117: Net-(J301-Pad117) -> /exp/UART3_RX
- J301 pad 165: BT81X.GPIO0 -> /exp/POWER
- J301 pad 7: ESP32.IO36 -> ESP32.IO26
- J301 pad 76: iMX8.GPIO3.IO7 -> Net-(J301-Pad76)
- J303 pad 1: GND -> Net-(J303-Pad1)
- J4 pad 4: /SPK_L+ -> Net-(J4-Pad4)
- J4 pad 5: /SPK_L_HP+ -> Net-(J4-Pad5)
- J4 pad 6: Net-(C39-Pad2) -> Net-(J4-Pad6)
- J4 pad 7: /SPK_R+ -> Net-(J4-Pad7)
- J4 pad 8: /SPK_R_HP_+ -> Net-(J4-Pad8)
- J4 pad 9: Net-(C38-Pad2) -> Net-(J4-Pad9)
- L1 pad 1: Net-(C1-Pad1) -> /BQ_SW
- R15 pad 2: GND -> +3V3
- R2 pad 1: Net-(C5-Pad1) -> Net-(C3-Pad1)
- R26 pad 1: Net-(R26-Pad1) -> BT81X.GPIO2
- R26 pad 2: /SPK_EN -> +3V3
- R3 pad 1: Net-(R3-Pad1) -> Net-(R2-Pad2)
- R3 pad 2: Net-(D1-Pad1) -> GND
- R31 pad 1: +VSYS -> VDDA
- R31 pad 2: Net-(R32-Pad2) -> Net-(R31-Pad2)
- R32 pad 1: Net-(R33-Pad1) -> Net-(R32-Pad1)
- R4 pad 1: Net-(R2-Pad2) -> Net-(R4-Pad1)
- R4 pad 2: GND -> Net-(D2-Pad1)
- U1 pad 38: /DISP_DE_INV -> /DISP_DE
- U13 pad 10: /SPK_L- -> /AUDIO_OUT_L-
- U13 pad 4: Net-(R26-Pad1) -> /SPK_EN
- U13 pad 7: +VSYS -> VDDA
- U13 pad 8: +VSYS -> VDDA
- U13 pad 9: /SPK_L_HP+ -> /AUDIO_OUT_L+
- U14 pad 10: /SPK_R- -> /AUDIO_OUT_R-
- U14 pad 7: +VSYS -> VDDA
- U14 pad 8: +VSYS -> VDDA
- U14 pad 9: /SPK_R_HP_+ -> /AUDIO_OUT_R+
- U18 pad 1: Net-(R32-Pad2) -> /SPK_GAIN_SEL
- U18 pad 2: GND -> VDDA
- U18 pad 3: Net-(R33-Pad1) -> GND
- U18 pad 4: /SPK_GAIN -> Net-(R32-Pad1)
- U18 pad 5: +VSYS -> /SPK_GAIN
- U18 pad 6: /SPK_GAIN_SEL -> Net-(R31-Pad2)
- U201 pad 10: Net-(U201-Pad10) -> BQ.INT
- U201 pad 11: Net-(U201-Pad11) -> ESP32.IO26
- U201 pad 4: ESP32.IO36 -> Net-(U201-Pad4)
- U403 pad 26: /disp/BT81X_AUDIO -> BT81X.AUDIO
- U407 pad 1: +VCTP -> TMUX.I2C0.SCL
- U407 pad 10: iMX8.GPIO5.IO29 -> /disp/CTP_RST
- U407 pad 11: iMX8.GPIO5.IO28 -> TMUX.GPIO0
- U407 pad 12: iMX8.I2C3.SDA -> iMX8.GPIO5.IO29
- U407 pad 13: iMX8.I2C3.SCL -> GND
- U407 pad 15: GND -> BT81X.DISP
- U407 pad 3: /disp/CTP_SDA -> iMX8.I2C3.SDA
- U407 pad 4: /disp/CTP_INT -> TMUX.I2C0.SDA
- U407 pad 5: /disp/CTP_RST -> /disp/CTP_SDA
- U407 pad 6: Net-(U407-Pad6) -> GND
- U407 pad 7: GND -> /disp/CTP_INT
- U407 pad 8: /disp/iMX8_CTP_EN -> TMUX.GPIO1
- U407 pad 9: Net-(U407-Pad9) -> iMX8.GPIO5.IO28
Routing:
- net BQ.INT: track 0.00 -> 181.9 mm, vias 0 -> 4
- net BT81X.AUDIO: track 0.00 -> 83.4 mm, vias 0 -> 2
- net /exp/POWER: track 0.00 -> 81.1 mm, vias 0 -> 2
- net ESP32.IO36: track 69.1 -> 0.00 mm, vias 2 -> 0
- net ESP32.IO26: track 0.00 -> 57.6 mm, vias 0 -> 2
- net /disp/iMX8_CTP_EN: track 53.4 -> 0.00 mm, vias 5 -> 0
- net BT81X.CTP.RST: track 49.0 -> 0.00 mm
- net BT81X.GPIO2: track 74.4 -> 123.0 mm, vias 4 -> 7
- net BT81X.CTP.INT: track 47.6 -> 0.00 mm
- net BT81X.CTP.SCL: track 45.6 -> 0.00 mm
- net BT81X.CTP.SDA: track 45.6 -> 0.00 mm, vias 2 -> 0
- net /SPK_EN: track 40.3 -> 81.4 mm, vias 4 -> 8
- net TMUX.GPIO1: track 32.7 -> 65.4 mm, vias 4 -> 3
- net TMUX.GPIO0: track 40.0 -> 71.3 mm, vias 4 -> 3
- net WAKE: track 117.8 -> 147.6 mm, vias 6 -> 7
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- added copper zone on PWR, net /BQ_PMID
- added copper zone on F.Cu, net /BQ_SW
- added copper zone on B.Cu, net DISP_LED_A
- added copper zone on F.Cu, net VDD
- added copper zone on F.Cu, net VDDA
- added copper zone on PWR, net VDDA
- removed copper zone on F.Cu, net /SPK_L_HP+
- removed copper zone on F.Cu, net /SPK_R_HP_+
- removed copper zone on B.Cu, net DISP_LED_K
- removed copper zone on F.Cu, net Net-(C1-Pad1)
Other:
- outline, holes or cut-outs redrawn
- board text added: "+3.3V"
- board text added: "CS"
- board text added: "GND"
- board text added: "GPIO0"
- board text added: "IO0"
- board text added: "IO1"
- board text added: "IO2"
- board text added: "IO3"
- board text added: "MISO"
- board text added: "MOSI"
- board text added: "RX"
- board text added: "SCK"
- board text added: "SCL"
- board text added: "SDA"
- board text added: "TX"
