File: hw/rvPhone/disp.sch (KiCad schematic (older format))
At the start: 73 parts, among them J401 Touch, J402 Display, U401 FAN5333BSX, U402 SN74LVC3G06DCU, U403 BT815Q, U404 IS25LP128-JKLE, U405 DS90C185, U406 TS3DV520E, U407 TXS0104ERGY, U408 TXS0104ERGY, U409 SN74LVC2G06DRY, Y401 12MHz

Commit message: rev2 board
Parts:
- removed C405, C407: 27pF, Capacitor_SMD:C_0603_1608Metric, symbol Device:C
- removed JP401: CTP_PWR, Jumper:SolderJumper-3_P1.3mm_Open_RoundedPad1.0x1.5mm, symbol Device:Jumper_NC_Dual
- removed R414: 10K, Resistor_SMD:R_0603_1608Metric, symbol Device:R
- removed R417: 100K, Resistor_SMD:R_0603_1608Metric, symbol Device:R
- removed U403: BT815Q, Package_DFN_QFN:QFN-64-1EP_9x9mm_P0.5mm_EP7.3x7.3mm_ThermalVias, symbol ft81x:BT815Q
- removed U406: TS3DV520E, footprints:Texas_R-PWQFN-N42, symbol ts:TS3DV520E
- removed U409: SN74LVC2G06DRY, footprints:USON-6_1.45x1mm_P0.5mm, symbol sn74:SN74LVC2G06DRY
- added C441: 10uF, Capacitor_SMD:C_0603_1608Metric, symbol Device:C
- added JP401: CTP_PWR, Jumper:SolderJumper-3_P1.3mm_Open_RoundedPad1.0x1.5mm, symbol Jumper:SolderJumper_3_Open
- added JP402: VOD_SEL, Jumper:SolderJumper-3_P1.3mm_Open_RoundedPad1.0x1.5mm, symbol Device:Jumper_NC_Dual
- added R418: 100K, Resistor_SMD:R_0603_1608Metric, symbol Device:R
- added TP401: AUDIO, TestPoint:TestPoint_Pad_D1.5mm, symbol Connector:TestPoint
- added U403: BT817Q, Package_DFN_QFN:QFN-64-1EP_9x9mm_P0.5mm_EP6x6mm_ThermalVias, symbol ftdi:BT817Q
- added U406: TS3DV520ERUA, footprints:Texas_R-PWQFN-N42, symbol ts:TS3DV520ERUA
- added U409: SN74LVC2G06DCK, Package_TO_SOT_SMD:Texas_R-PDSO-G6, symbol sn74:SN74LVC2G06DCK
- C409, C410: value 18pF -> 10pF
- R405: value R -> 68R
- R414: renamed from R415; value 1K -> R
- R415: renamed from R416; value 1K -> R
Connections:
- net +1V8: now also C441.2, JP401.1 (A), JP402.1, U403.28 (VCCIO2), U409.5 (VCC); no longer C427.1, C428.1, C429.1, C430.1, C431.1, C432.1, C433.1
- net +3V3: now also C427.1, C428.1, C429.1, C430.1, C431.1, C432.1, C433.1, JP401.3 (B), U403.17 (VCCIO3), U403.24 (VCC), U403.27 (VCCA), U403.9 (VCCIO1), U406.1 (VCC), U406.13 (VCC), U406.22 (VCC), U406.31 (VCC), U406.4 (VCC), U406.40 (VCC), U406.7 (VCC); no longer C439.1, J401.3 (Pin_3), R414.1, R415.1
- net +VCTP: now also C439.1, J401.3 (Pin_3), R414.1, R415.1, JP401.2 (C)
- net BT81X.B0: now also U403.47 (B0)
- net BT81X.B1: now also U403.46 (B1)
- net BT81X.B2: now also U403.45 (B2)
- net BT81X.B3: now also U403.44 (B3)
- net BT81X.B4: now also U403.43 (B4)
- net BT81X.B5: now also U403.42 (B5)
- net BT81X.B6: now also U403.41 (B6)
- net BT81X.B7: now also U403.40 (B7)
- net BT81X.BL_PWM: now also U403.34 (BL_PWM)
- net BT81X.CTP.INT: now also U403.30 (CTP_INT_N)
- net BT81X.CTP.RST: now also U403.29 (CTP_RST_N)
- net BT81X.CTP.SCL: now also U403.31 (CTP_SCL)
- net BT81X.CTP.SDA: now also U403.32 (CTP_SDA)
- net BT81X.DE: now also U403.35 (DE)
- net BT81X.DISP: now also U403.38 (DISP), U406.12 (SEL), U409.1 (1A)
- net BT81X.G0: now also U403.56 (G0)
- net BT81X.G1: now also U403.55 (G1)
- net BT81X.G2: now also U403.54 (G2)
- net BT81X.G3: now also U403.53 (G3)
- net BT81X.G4: now also U403.52 (G4)
- net BT81X.G5: now also U403.51 (G5)
- net BT81X.G6: now also U403.50 (G6)
- net BT81X.G7: now also U403.49 (G7)
- net BT81X.GPIO0: now also U403.7 (GPIO0/IO2)
- net BT81X.GPIO1: now also R418.1, U403.8 (GPIO1/IO3)
- net BT81X.GPIO2: now also U403.10 (GPIO2)
- net BT81X.GPIO3: now also U403.13 (GPIO3)
- net BT81X.HSYNC: now also U403.37 (HSYNC)
- net BT81X.PCLK: now also U403.39 (PCLK)
- net BT81X.R0: now also U403.1 (R0)
- net BT81X.R1: now also U403.64 (R1)
- net BT81X.R2: now also U403.63 (R2)
- net BT81X.R3: now also U403.62 (R3)
- net BT81X.R4: now also U403.61 (R4)
- net BT81X.R5: now also U403.60 (R5)
- net BT81X.R6: now also U403.59 (R6)
- net BT81X.R7: now also U403.58 (R7)
- net BT81X.VSYNC: now also U403.36 (VSYNC)
- net BT81X_1V2: now also U403.2 (VIN1V2), U403.25 (VOUT1V2), U403.57 (VIN1V2)
- net BT81X_QSPI_CLK: now also U403.14 (SPIMSCK)
- net BT81X_QSPI_CS: now also U403.15 (SPIMCS)
- net BT81X_QSPI_DQ_0: now also U403.16 (SPIMMOSI)
- net BT81X_QSPI_DQ_1: now also U403.18 (SPIMMISO)
- net BT81X_QSPI_DQ_2: now also U403.19 (SPIMIO2)
- net BT81X_QSPI_DQ_3: now also U403.20 (SPIMIO3)
- net BT81X_X1: now also U403.21 (X1/CLK)
- net BT81X_X2: now also U403.22 (X2)
- net DISP_CS: now also J402.19 (Pin_19); no longer J402.22 (Pin_22)
- net DISP_LVDS_A0N: now also U406.15 (A9)
- net DISP_LVDS_A0P: now also U406.14 (A8)
- net DISP_LVDS_A1N: now also U406.11 (A7)
- net DISP_LVDS_A1P: now also U406.10 (A6)
- net DISP_LVDS_A2N: now also U406.9 (A5)
- net DISP_LVDS_A2P: now also U406.8 (A4)
- net DISP_LVDS_A3N: now also U406.3 (A1)
- net DISP_LVDS_A3P: now also U406.2 (A0)
- net GND: now also C441.1, JP402.3, R418.2, U403.23 (GND), U403.33 (GND), U403.48 (GND), U403.65 (EP), U406.43 (GND), U409.2 (GND)
- net GPIO_0: now also U403.11 (INT_N)
- net SPI1.MISO: now also J402.22 (Pin_22), U403.4 (MISO/IO1); no longer J402.19 (Pin_19)
- net SPI1.MOSI: now also J402.21 (Pin_21), U403.5 (MOSI/IO0); no longer J402.20 (Pin_20)
- net SPI1.SCK: now also J402.20 (Pin_20), U403.3 (SCK); no longer J402.21 (Pin_21)
- net SPI1.SS2: now also U403.6 (CS_N)
- net iMX8_CTP_EN: now also U409.4 (2Y), U409.6 (1Y)
- net at U405.39 (VOD_SEL): now also JP402.2
- net at C408.1, R406.2: now also U403.12 (PD_N)
- net DISP_LVDS_CLK_N renamed DISP_LVDS_CLKN
- net DISP_LVDS_CLKN: now also U406.6 (A3)
- net DISP_LVDS_CLK_P renamed DISP_LVDS_CLKP
- net DISP_LVDS_CLKP: now also U406.5 (A2)
- net DS90_LVDS_A0_N renamed DS90_LVDS_A0N
- net DS90_LVDS_A0N: now also U406.21 (9B2)
- net DS90_LVDS_A0_P renamed DS90_LVDS_A0P
- net DS90_LVDS_A0P: now also U406.20 (8B2)
- net DS90_LVDS_A1_N renamed DS90_LVDS_A1N
- net DS90_LVDS_A1N: now also U406.23 (7B2)
- net DS90_LVDS_A1_P renamed DS90_LVDS_A1P
- net DS90_LVDS_A1P: now also U406.24 (6B2)
- net DS90_LVDS_A2_N renamed DS90_LVDS_A2N
- net DS90_LVDS_A2N: now also U406.27 (5B2)
- net DS90_LVDS_A2_P renamed DS90_LVDS_A2P
- net DS90_LVDS_A2P: now also U406.28 (4B2)
- net DS90_LVDS_A3_N renamed DS90_LVDS_A3N
- net DS90_LVDS_A3N: now also U406.36 (1B2)
- net DS90_LVDS_A3_P renamed DS90_LVDS_A3P
- net DS90_LVDS_A3P: now also U406.37 (0B2)
- net DS90_LVDS_CLK_N renamed DS90_LVDS_CLKN
- net DS90_LVDS_CLKN: now also U406.32 (3B2)
- net DS90_LVDS_CLK_P renamed DS90_LVDS_CLKP
- net DS90_LVDS_CLKP: now also U406.33 (2B2)
- net iMX8.GPIO3.IO11 renamed iMX8.GPIO5.IO29
- net iMX8.GPIO3.IO12 renamed iMX8.GPIO5.IO28
- net iMX8.GPIO3.IO13 renamed iMX8.GPIO3.IO7
- net iMX8.GPIO3.IO7: now also U409.3 (2A)
- net iMX8.I2C1.SCL renamed iMX8.I2C3.SCL
- net iMX8.I2C1.SDA renamed iMX8.I2C3.SDA
- new net: TP401.1, U403.26 (AUDIO_L)
- new net iMX8.LVDS0.A0N: U406.18 (9B1)
- new net iMX8.LVDS0.A0P: U406.16 (8B1)
- new net iMX8.LVDS0.A1N: U406.25 (7B1)
- new net iMX8.LVDS0.A1P: U406.26 (6B1)
- new net iMX8.LVDS0.A2N: U406.29 (5B1)
- new net iMX8.LVDS0.A2P: U406.30 (4B1)
- new net iMX8.LVDS0.A3N: U406.38 (1B1)
- new net iMX8.LVDS0.A3P: U406.39 (0B1)
- new net iMX8.LVDS0.CLKN: U406.34 (3B1)
- new net iMX8.LVDS0.CLKP: U406.35 (2B1)
- no-connect marks 6 -> 4
Other:
- moved on the sheet: C401, C402, C403, C404, C406, C421, C422, C423, C424, C425, C426, C427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

Commit message: temp commit for merge
Parts:
- removed C435, C436, C437, C438, C439, C440: 0.1uF, Capacitor_SMD:C_0603_1608Metric, symbol Device:C
- removed J401: Touch, Connector_FFC-FPC:Hirose_FH12-8S-0.5SH_1x08-1MP_P0.50mm_Horizontal, symbol Connector_Generic:Conn_01x08
- removed J402: Display, Connector_FFC-FPC:Hirose_FH12-26S-0.5SH_1x26-1MP_P0.50mm_Horizontal, symbol Connector_Generic:Conn_01x26
- removed JP401: CTP_PWR, Jumper:SolderJumper-3_P1.3mm_Open_RoundedPad1.0x1.5mm, symbol Jumper:SolderJumper_3_Open
- removed R412, R413: 47K, Resistor_SMD:R_0603_1608Metric, symbol Device:R
- removed R414, R415: R, Resistor_SMD:R_0603_1608Metric, symbol Device:R
- removed U407, U408: TXS0104ERGY, Package_DFN_QFN:Texas_S-PVQFN-N14_ThermalVias, symbol tx:TXS0104ERGY
- removed U409: SN74LVC2G06DCK, Package_TO_SOT_SMD:Texas_R-PDSO-G6, symbol sn74:SN74LVC2G06DCK
- added J401: Display, Connector_Molex:Molex_SlimStack_54722-0304_2x15_P0.50mm_Vertical, symbol Connector_Generic:Conn_02x15_Odd_Even
- added J402, J403: Spacer, footprints:Spacer, symbol myConn:Spacer
- added U407: TMUX1574RSV, footprints:UQFN-16_1.8x2.6mm_P0.4mm, symbol tmux:TMUX1574RSV
- L401: footprint footprints:L_Murata_LQH66SN -> footprints:Murata-LQH66SN
Connections:
- net labels added: BT81X_AUDIO, GPIO_23, SPI1.SS3, TMUX.GPIO0, TMUX.GPIO1, TMUX.I2C0.SCL, TMUX.I2C0.SDA
- net labels removed: +VCTP, GPIO_0, SPI1.SS2, iMX8.GPIO3.IO7, iMX8_CTP_EN
- wire segments 518 -> 449
- no-connect marks 4 -> 8
Other:
- moved on the sheet: C406, C434, R403, R404, R405, R418, TP401

Commit message: HW REV 3.0
Parts:
- removed TP401: AUDIO, TestPoint:TestPoint_Pad_D1.5mm, symbol Connector:TestPoint
Connections:
- net labels added: BT81X.AUDIO
- net labels removed: BT81X_AUDIO
- wire segments 449 -> 447
Changed lines of the file:
@@
 Text GLabel 8300 5700 0    55   Input ~ 0
 iMX8.I2C3.SCL
-Text GLabel 2250 9350 0    55   BiDi ~ 0
+Text GLabel 5750 6900 0    55   BiDi ~ 0
 BT81X.CTP.INT
-Text GLabel 2250 9250 0    55   BiDi ~ 0
+Text GLabel 5750 6800 0    55   BiDi ~ 0
 BT81X.CTP.SDA
-Text GLabel 2250 9150 0    55   Input ~ 0
+Text GLabel 5750 6700 0    55   Input ~ 0
 BT81X.CTP.SCL
-Text GLabel 2250 9450 0    55   Input ~ 0
+Text GLabel 5750 7000 0    55   Input ~ 0
 BT81X.CTP.RST
 NoConn ~ 8350 4300
@@
 	1    0    0    -1
 $EndComp
-$Comp
-L Connector:TestPoint TP401
-U 1 1 6100EDA6
-P 900 8000
-F 0 "TP401" H 650 8050 50  0000 L CNN
-F 1 "AUDIO" H 750 8200 50  0000 L CNN
-F 2 "TestPoint:TestPoint_Pad_D1.5mm" H 1100 8000 50  0001 C CNN
-F 3 "~" H 1100 8000 50  0001 C CNN
-	1    900  8000
-	1    0    0    -1
-$EndComp
-Wire Wire Line
-	1550 4800 2150 4800
 $Comp
 L power:+3.3V #PWR0128
@@
 	14000 6250 14000 6850
 Connection ~ 14000 6850
-Text Label 1550 4800 0    60   ~ 0
-BT81X_AUDIO
-Text Label 1550 8050 2    60   ~ 0
-BT81X_AUDIO
-Wire Wire Line
-	1550 8050 900  8050
-Wire Wire Line
-	900  8050 900  8000
 Wire Wire Line
 	13750 7450 13750 7500
@@
 Wire Wire Line
 	9500 6700 9500 6800
-NoConn ~ 2250 9150
-NoConn ~ 2250 9250
-NoConn ~ 2250 9350
-NoConn ~ 2250 9450
+NoConn ~ 5750 6700
+NoConn ~ 5750 6800
+NoConn ~ 5750 6900
+NoConn ~ 5750 7000
 Text Label 10400 5900 2    55   ~ 0
 CTP_SCL
@@
 U 1 1 6135689D
 P 8950 6050
+AR Path="/6135689D" Ref="U407"  Part="1"
+AR Path="/5FC4BBBD/6135689D" Ref="U407"  Part="1"
 F 0 "U407" H 8950 6500 60  0000 C CNN
 F 1 "TMUX1574RSV" H 8950 5300 60  0000 C CNN
@@
 	-1   0    0    -1
 $EndComp
+Text GLabel 1850 4800 0    60   Output ~ 0
+BT81X.AUDIO
+Wire Wire Line
+	2150 4800 1850 4800
 $EndSCHEMATC

Commit message: added pull-up pull-dn resistors; fixed input power;
Parts:
- removed R418: 100K, Resistor_SMD:R_0603_1608Metric, symbol Device:R
Connections:
- wire segments 447 -> 442
Changed lines of the file:
@@
 Wire Wire Line
 	3200 1800 3800 1800
-Text GLabel 9850 6400 2    55   Input ~ 0
+Text GLabel 9900 6400 2    55   Input ~ 0
 BT81X.DISP
 Text GLabel 13000 2300 2    55   Input ~ 0
@@
 F 3 "" H 7250 1450 50  0001 C CNN
 	1    7250 1450
-	1    0    0    -1
-$EndComp
-$Comp
-L Device:R R418
-U 1 1 6026DA78
-P 13750 7300
-F 0 "R418" V 13850 7300 50  0000 C CNN
-F 1 "100K" V 13750 7300 50  0000 C CNN
-F 2 "Resistor_SMD:R_0603_1608Metric" V 13680 7300 50  0001 C CNN
-F 3 "~" H 13750 7300 50  0001 C CNN
-	1    13750 7300
 	1    0    0    -1
 $EndComp
@@
 	13650 6650 14100 6650
 Wire Wire Line
-	13650 6750 13750 6750
-Wire Wire Line
 	13650 6950 14100 6950
 $Comp
@@
 Wire Wire Line
 	14100 6850 14000 6850
-Wire Wire Line
-	14000 6850 14000 7500
 $Comp
 L power:+3.3V #PWR0176
@@
 Connection ~ 14000 6850
 Wire Wire Line
-	13750 7450 13750 7500
-Wire Wire Line
-	13750 7500 14000 7500
-Connection ~ 14000 7500
-Wire Wire Line
-	14000 7500 14000 7550
-Wire Wire Line
 	13650 7050 14100 7050
-Wire Wire Line
-	13750 7150 13750 6750
-Connection ~ 13750 6750
-Wire Wire Line
-	13750 6750 14100 6750
 NoConn ~ 14600 5650
 Wire Wire Line
@@
 	10400 6200 9450 6200
 Wire Wire Line
-	9850 6400 9450 6400
+	9900 6400 9450 6400
 Wire Wire Line
 	9450 6500 9500 6500
@@
 Wire Wire Line
 	2150 4800 1850 4800
+Wire Wire Line
+	13650 6750 14100 6750
+Wire Wire Line
+	14000 6850 14000 7550
 $EndSCHEMATC

Commit message: REV3.1:  - fixed audio  - added spacers  - UART is routed through audio mux instead of I2C  - proper display connector alignment
Parts:
- removed R408: 47K, Resistor_SMD:R_0603_1608Metric, symbol Device:R
- added J403: Spacer, footprints:Spacer_small, symbol myConn:Spacer
- J402: footprint footprints:Spacer -> footprints:Spacer_small
- J404: renamed from J403; footprint footprints:Spacer -> footprints:Spacer_small
- JP402: footprint Jumper:SolderJumper-3_P1.3mm_Open_RoundedPad1.0x1.5mm -> Jumper:SolderJumper-3_P1.3mm_Bridged2Bar12_RoundedPad1.0x1.5mm
- renumbered R409 to R408, R410 to R409, R411 to R410
Connections:
- net labels added: BT81X.INT, CTP.RST, I2C0.SCL, I2C0.SDA
- net labels removed: BT81X.CTP.INT, BT81X.CTP.RST, BT81X.CTP.SCL, BT81X.CTP.SDA, TMUX.GPIO0, TMUX.GPIO1, TMUX.I2C0.SCL, TMUX.I2C0.SDA
- wire segments 442 -> 436
