File: hw/rvPhone/exp.sch (KiCad schematic (older format))
At the start: 56 parts, among them J301 iMX8, J302 Touch, J303 Display, J304 Prog, U301 SN65LVDS822_SWAP, U302 TS3DDR3812, U303 TS3DDR3812, U304 TS3DDR3812

Commit message: stereo audio out; lvds display; LSM9DS1 added
Parts:
- removed C319, C321, C325, C327, C337, C339: 1uF, Capacitor_SMD:C_0603_1608Metric, symbol Device:C_Small
- removed C320, C322, C323, C326, C328, C329, C331, C333, C335, C338, C340: 0.1uF, Capacitor_SMD:C_0603_1608Metric, symbol Device:C_Small
- removed C324, C330, C332, C334, C336: 0.01uF, Capacitor_SMD:C_0603_1608Metric, symbol Device:C_Small
- removed C341, C342: 0.1uF, Capacitor_SMD:C_0603_1608Metric, symbol Device:C
- removed J301: iMX8, footprints:Socket_SODIMM_DDR3_TE_2013289, symbol SODIMM-204:iMX8
- removed J302: Touch, Connector_FFC-FPC:Hirose_FH12-6S-0.5SH_1x06-1MP_P0.50mm_Horizontal, symbol Connector_Generic:Conn_01x06
- removed J303: Display, Connector_FFC-FPC:Hirose_FH12-40S-0.5SH_1x40-1MP_P0.50mm_Horizontal, symbol Connector_Generic:Conn_01x40
- removed R301: 4.7K, Resistor_SMD:R_0603_1608Metric, symbol Device:R
- removed R302, R303: 1K, Resistor_SMD:R_0603_1608Metric, symbol Device:R
- removed R304, R306: 100K, Resistor_SMD:R_0603_1608Metric, symbol Device:R
- removed R305: 47K, Resistor_SMD:R_0603_1608Metric, symbol Device:R
- removed U301: SN65LVDS822_SWAP, Package_DFN_QFN:QFN-48-1EP_7x7mm_P0.5mm_EP5.15x5.15mm_ThermalVias, symbol sn65:SN65LVDS822_SWAP
- removed U302, U303, U304: TS3DDR3812, footprints:Texas_R-PWQFN-N42, symbol ts3ddr:TS3DDR3812
- added J301: iMX8, footprints:Socket_SODIMM_DDR3_TE_2013289, symbol myConn:iMX8
- renumbered J304 to J302
Connections:
- net +VSYS: now also J301.10 (PIN10), J301.114 (PIN114), J301.132 (PIN132), J301.150 (PIN150), J301.168 (PIN168), J301.186 (PIN186), J301.204 (PIN204), J301.28 (PIN28), J301.46 (PIN46), J301.64 (PIN64), J301.78 (PIN78), J301.96 (PIN96)
- net ESP32.HSPI.MISO: now also J301.15 (PIN15)
- net ESP32.HSPI.MOSI: now also J301.11 (PIN11)
- net ESP32.HSPI.SCK: now also J301.13 (PIN13)
- net ESP32.HSPI.SS0: now also J301.17 (PIN17)
- net ESP32.IO27: now also J301.9 (PIN9)
- net ESP32.IO36: now also J301.7 (PIN7)
- net GND: now also J301.1 (PIN1), J301.105 (PIN105), J301.123 (PIN123), J301.141 (PIN141), J301.159 (PIN159), J301.177 (PIN177), J301.19 (PIN19), J301.37 (PIN37), J301.55 (PIN55), J301.71 (PIN71), J301.87 (PIN87)
- net at C301.1: now also J301.183 (PIN183)
- net TPS.VOUT: no longer names the net of J302.12 (Pin_12)
- new net iMX8.GPIO3.IO11: J301.153 (PIN153)
- new net iMX8.GPIO3.IO12: J301.151 (PIN151)
- new net iMX8.GPIO3.IO13: J301.149 (PIN149)
- new net iMX8.I2C1.SCL: J301.129 (PIN129)
- new net iMX8.I2C1.SDA: J301.135 (PIN135)
- new net iMX8.LVDS0.A0_N: J301.41 (PIN41)
- new net iMX8.LVDS0.A0_P: J301.39 (PIN39)
- new net iMX8.LVDS0.A1_N: J301.47 (PIN47)
- new net iMX8.LVDS0.A1_P: J301.45 (PIN45)
- new net iMX8.LVDS0.A2_N: J301.53 (PIN53)
- new net iMX8.LVDS0.A2_P: J301.51 (PIN51)
- new net iMX8.LVDS0.A3_N: J301.59 (PIN59)
- new net iMX8.LVDS0.A3_P: J301.57 (PIN57)
- new net iMX8.LVDS0.CLK_N: J301.35 (PIN35)
- new net iMX8.LVDS0.CLK_P: J301.33 (PIN33)
- new net iMX8.PWM1: J301.75 (PIN75)
- new net iMX8.USB1.D_N: J301.178 (PIN178)
- new net iMX8.USB1.D_P: J301.176 (PIN176)
- no-connect marks 164 -> 158
Other:
- moved on the sheet: J302

Commit message: rev2 board
Parts:
- removed J302: Prog, Connector_FFC-FPC:Hirose_FH12-12S-0.5SH_1x12-1MP_P0.50mm_Horizontal, symbol Connector_Generic:Conn_01x12
- added C319: 0.1uF, Capacitor_SMD:C_0603_1608Metric, symbol Device:C
- added J305: Micro_SD_Card, footprints:microSD, symbol Connector:Micro_SD_Card
- added JP301: ALT_BOOT, Jumper:SolderJumper-2_P1.3mm_Open_RoundedPad1.0x1.5mm, symbol Device:Jumper_NC_Small
- C314, C315, C316, C317, C318: footprint Capacitor_SMD:C_0603_1608Metric -> Capacitor_SMD:C_0805_2012Metric
Connections:
- net GND: now also J301.61 (PIN61), J301.67 (PIN67), C319.2, J305.6 (VSS), J305.9 (SHIELD)
- net iMX8.PWM1: now also J301.200 (PIN200); no longer J301.75 (PIN75)
- net ALT_BOOT: now reaches J301.185 (PIN185)
- net ALT_BOOT: now also JP301.1
- net iMX8.GPIO5.IO29: now reaches J301.3 (PIN3)
- net iMX8.I2C3.SCL: now reaches J301.43 (PIN43)
- net iMX8.I2C3.SDA: now reaches J301.49 (PIN49)
- net iMX8.GPIO5.IO28: now reaches J301.5 (PIN5)
- net iMX8.GPIO3.IO7: now reaches J301.76 (PIN76)
- net SD2_CLK: now reaches J301.80 (PIN80)
- net SD2_CLK: now also J305.5 (CLK)
- net SD2_CMD: now reaches J301.82 (PIN82)
- net SD2_CMD: now also J305.3 (CMD)
- net SD2_DAT0: now reaches J301.84 (PIN84)
- net SD2_DAT0: now also J305.7 (DAT0)
- net SD2_DAT1: now reaches J301.86 (PIN86)
- net SD2_DAT1: now also J305.8 (DAT1)
- net SD2_DAT2: now reaches J301.88 (PIN88)
- net SD2_DAT2: now also J305.1 (DAT2)
- net SD2_DAT3: now reaches J301.90 (PIN90)
- net SD2_DAT3: now also J305.2 (DAT3/CD)
- net iMX8.GPIO3.IO11: no longer names the net of J301.153 (PIN153)
- net iMX8.GPIO3.IO12: no longer names the net of J301.151 (PIN151)
- net iMX8.GPIO3.IO13: no longer names the net of J301.149 (PIN149)
- net iMX8.I2C1.SCL: no longer names the net of J301.129 (PIN129)
- net iMX8.I2C1.SDA: no longer names the net of J301.135 (PIN135)
- net iMX8.LVDS0.A0_N renamed iMX8.LVDS0.A0N
- net iMX8.LVDS0.A0_P renamed iMX8.LVDS0.A0P
- net iMX8.LVDS0.A1_N renamed iMX8.LVDS0.A1N
- net iMX8.LVDS0.A1_P renamed iMX8.LVDS0.A1P
- net iMX8.LVDS0.A2_N renamed iMX8.LVDS0.A2N
- net iMX8.LVDS0.A2_P renamed iMX8.LVDS0.A2P
- net iMX8.LVDS0.A3_N renamed iMX8.LVDS0.A3N
- net iMX8.LVDS0.A3_P renamed iMX8.LVDS0.A3P
- net iMX8.LVDS0.CLK_N renamed iMX8.LVDS0.CLKN
- net iMX8.LVDS0.CLK_P renamed iMX8.LVDS0.CLKP
- new net +3V3: C319.1, J305.4 (VDD), JP301.2
- no-connect marks 158 -> 148
Other:
- moved on the sheet: C301

Commit message: temp commit for merge
Parts:
- removed J305: Micro_SD_Card, footprints:microSD, symbol Connector:Micro_SD_Card
- removed JP301: ALT_BOOT, Jumper:SolderJumper-2_P1.3mm_Open_RoundedPad1.0x1.5mm, symbol Device:Jumper_NC_Small
- added C320: 22uF, Capacitor_SMD:C_0805_2012Metric, symbol Device:C
- added J302: Micro_SD_Card_Det, footprints:Molex_MicroSD-5027740891, symbol Connector:Micro_SD_Card_Det
- added J303: Spacer, footprints:Spacer, symbol myConn:Spacer
- added JP301: USB_VBUS, Jumper:SolderJumper-2_P1.3mm_Open_RoundedPad1.0x1.5mm, symbol Jumper:SolderJumper_2_Open
- added JP302: USB_ID, Jumper:SolderJumper-2_P1.3mm_Open_RoundedPad1.0x1.5mm, symbol Jumper:SolderJumper_2_Open
- added R301: 100K, Resistor_SMD:R_0603_1608Metric, symbol Device:R
- added SW301: iMX8_ALT_BOOT, Button_Switch_SMD:SW_SPST_PTS810, symbol Switch:SW_Push
- added SW302: iMX8_RST, Button_Switch_SMD:SW_SPST_PTS810, symbol Switch:SW_Push
- added SW303: iMX8_PWR, Button_Switch_SMD:SW_SPST_PTS810, symbol Switch:SW_Push
- J301: footprint footprints:Socket_SODIMM_DDR3_TE_2013289 -> footprints:TE_SODIMMDDR3-2013289
Connections:
- net labels added: ESP32.IO26, POWER, RESET, SD2_DET, iMX8.USB1.ID, iMX8.USB1.VBUS
- net labels removed: ESP32.IO36, iMX8.GPIO3.IO7
- wire segments 178 -> 207
- no-connect marks 148 -> 145
Other:
- moved on the sheet: C319

Commit message: HW REV 3.0
Parts:
- removed J303: Spacer, footprints:Spacer, symbol myConn:Spacer
- added J303: Console, Connector_FFC-FPC:Hirose_FH12-6S-0.5SH_1x06-1MP_P0.50mm_Horizontal, symbol Connector_Generic:Conn_01x06
Connections:
- net labels added: UART3_RX, UART3_TX
- wire segments 207 -> 213
Changed lines of the file:
@@
 NoConn ~ 1500 6100
 NoConn ~ 1500 6200
-NoConn ~ 1500 6300
 NoConn ~ 1500 6400
 NoConn ~ 3000 5600
@@
 NoConn ~ 1500 6800
 NoConn ~ 1500 6700
-NoConn ~ 1500 6600
 NoConn ~ 1500 6500
 Text GLabel 1300 1300 0    55   BiDi ~ 0
@@
 Wire Wire Line
 	5450 6650 5550 6650
-$Comp
-L myConn:Spacer J303
-U 1 1 60E13E30
-P 7350 5050
-F 0 "J303" H 7300 5150 50  0000 L CNN
-F 1 "Spacer" H 7250 4950 50  0000 L CNN
-F 2 "footprints:Spacer" H 7350 5050 50  0001 C CNN
-F 3 "~" H 7350 5050 50  0001 C CNN
-	1    7350 5050
-	1    0    0    -1
-$EndComp
-$Comp
-L power:GND #PWR0182
-U 1 1 60E1444F
-P 7050 5150
-F 0 "#PWR0182" H 7050 4900 50  0001 C CNN
-F 1 "GND" H 7055 4977 50  0000 C CNN
-F 2 "" H 7050 5150 50  0001 C CNN
-F 3 "" H 7050 5150 50  0001 C CNN
-	1    7050 5150
-	1    0    0    -1
-$EndComp
-Wire Wire Line
-	7150 5050 7050 5050
-Wire Wire Line
-	7050 5050 7050 5150
 Wire Wire Line
 	1500 9000 600  9000
@@
 	5500 5800 4950 5800
 NoConn ~ 3000 4500
+$Comp
+L Connector_Generic:Conn_01x06 J303
+U 1 1 61AE2880
+P 8100 6400
+F 0 "J303" H 8050 6700 50  0000 L CNN
+F 1 "Console" H 7950 6000 50  0000 L CNN
+F 2 "Connector_FFC-FPC:Hirose_FH12-6S-0.5SH_1x06-1MP_P0.50mm_Horizontal" H 8100 6400 50  0001 C CNN
+F 3 "~" H 8100 6400 50  0001 C CNN
+	1    8100 6400
+	1    0    0    -1
+$EndComp
+$Comp
+L power:GND #PWR0184
+U 1 1 61AF1021
+P 7800 6800
+F 0 "#PWR0184" H 7800 6550 50  0001 C CNN
+F 1 "GND" H 7805 6627 50  0000 C CNN
+F 2 "" H 7800 6800 50  0001 C CNN
+F 3 "" H 7800 6800 50  0001 C CNN
+	1    7800 6800
+	1    0    0    -1
+$EndComp
+Wire Wire Line
+	7900 6700 7800 6700
+Wire Wire Line
+	7800 6700 7800 6800
+Wire Wire Line
+	7900 6600 7800 6600
+Wire Wire Line
+	7800 6600 7800 6700
+Connection ~ 7800 6700
+Text Label 600  6600 0    60   ~ 0
+UART3_RX
+Wire Wire Line
+	600  6600 1500 6600
+Text Label 600  6300 0    60   ~ 0
+UART3_TX
+Wire Wire Line
+	600  6300 1500 6300
+Text Label 7000 6400 0    60   ~ 0
+UART3_RX
+Wire Wire Line
+	7000 6400 7900 6400
+Text Label 7000 6500 0    60   ~ 0
+UART3_TX
+Wire Wire Line
+	7000 6500 7900 6500
+NoConn ~ 7900 6200
+NoConn ~ 7900 6300
 $EndSCHEMATC

Commit message: added pull-up pull-dn resistors; fixed input power;
Parts:
- added R302, R303: 10K, Resistor_SMD:R_0603_1608Metric, symbol Device:R
- added R304, R305: 47K, Resistor_SMD:R_0603_1608Metric, symbol Device:R
- added R306, R307: 100K, Resistor_SMD:R_0603_1608Metric, symbol Device:R
- R301: value 100K -> 47K
Connections:
- wire segments 213 -> 231
Other:
- moved on the sheet: J303
Changed lines of the file:
@@
 U 1 1 60F1E778
 P 5300 2250
-F 0 "R301" V 5400 2150 50  0000 L CNN
-F 1 "100K" V 5300 2150 50  0000 L CNN
+F 0 "R301" V 5400 2250 50  0000 C CNN
+F 1 "47K" V 5300 2250 50  0000 C CNN
 F 2 "Resistor_SMD:R_0603_1608Metric" V 5230 2250 50  0001 C CNN
 F 3 "~" H 5300 2250 50  0001 C CNN
@@
 L Connector_Generic:Conn_01x06 J303
 U 1 1 61AE2880
-P 8100 6400
-F 0 "J303" H 8050 6700 50  0000 L CNN
-F 1 "Console" H 7950 6000 50  0000 L CNN
-F 2 "Connector_FFC-FPC:Hirose_FH12-6S-0.5SH_1x06-1MP_P0.50mm_Horizontal" H 8100 6400 50  0001 C CNN
-F 3 "~" H 8100 6400 50  0001 C CNN
-	1    8100 6400
+P 5950 9550
+F 0 "J303" H 5850 9850 50  0000 L CNN
+F 1 "Console" H 5800 9150 50  0000 L CNN
+F 2 "Connector_FFC-FPC:Hirose_FH12-6S-0.5SH_1x06-1MP_P0.50mm_Horizontal" H 5950 9550 50  0001 C CNN
+F 3 "~" H 5950 9550 50  0001 C CNN
+	1    5950 9550
 	1    0    0    -1
 $EndComp
@@
 L power:GND #PWR0184
 U 1 1 61AF1021
-P 7800 6800
-F 0 "#PWR0184" H 7800 6550 50  0001 C CNN
-F 1 "GND" H 7805 6627 50  0000 C CNN
-F 2 "" H 7800 6800 50  0001 C CNN
-F 3 "" H 7800 6800 50  0001 C CNN
-	1    7800 6800
-	1    0    0    -1
-$EndComp
-Wire Wire Line
-	7900 6700 7800 6700
-Wire Wire Line
-	7800 6700 7800 6800
-Wire Wire Line
-	7900 6600 7800 6600
-Wire Wire Line
-	7800 6600 7800 6700
-Connection ~ 7800 6700
+P 5650 9950
+F 0 "#PWR0184" H 5650 9700 50  0001 C CNN
+F 1 "GND" H 5655 9777 50  0000 C CNN
+F 2 "" H 5650 9950 50  0001 C CNN
+F 3 "" H 5650 9950 50  0001 C CNN
+	1    5650 9950
+	1    0    0    -1
+$EndComp
+Wire Wire Line
+	5750 9850 5650 9850
+Wire Wire Line
+	5650 9850 5650 9950
+Wire Wire Line
+	5750 9750 5650 9750
+Wire Wire Line
+	5650 9750 5650 9850
+Connection ~ 5650 9850
 Text Label 600  6600 0    60   ~ 0
 UART3_RX
@@
 Wire Wire Line
 	600  6300 1500 6300
-Text Label 7000 6400 0    60   ~ 0
+Text Label 4850 9550 0    60   ~ 0
 UART3_RX
 Wire Wire Line
-	7000 6400 7900 6400
-Text Label 7000 6500 0    60   ~ 0
+	4850 9550 5750 9550
+Text Label 4850 9650 0    60   ~ 0
 UART3_TX
 Wire Wire Line
-	7000 6500 7900 6500
-NoConn ~ 7900 6200
-NoConn ~ 7900 6300
+	4850 9650 5750 9650
+NoConn ~ 5750 9350
+NoConn ~ 5750 9450
+Text GLabel 5450 8150 0    55   BiDi ~ 0
+ESP32.HSPI.SS0
+Text GLabel 5450 7750 0    55   Input ~ 0
+iMX8.I2C3.SCL
+Text GLabel 5450 7950 0    55   BiDi ~ 0
+iMX8.I2C3.SDA
+Text GLabel 5450 8550 0    55   Input ~ 0
+iMX8.PWM1
+Text GLabel 5450 8750 0    55   BiDi ~ 0
+iMX8.GPIO5.IO29
+Text GLabel 5450 8350 0    55   BiDi ~ 0
+iMX8.GPIO5.IO28
+$Comp
+L Device:R R302
+U 1 1 6291BF3B
+P 5700 7750
+F 0 "R302" V 5800 7750 50  0000 C CNN
+F 1 "10K" V 5700 7750 50  0000 C CNN
+F 2 "Resistor_SMD:R_0603_1608Metric" V 5630 7750 50  0001 C CNN
+F 3 "~" H 5700 7750 50  0001 C CNN
+	1    5700 7750
+	0    1    1    0
+$EndComp
+$Comp
+L Device:R R303
+U 1 1 6291C716
+P 5700 7950
+F 0 "R303" V 5800 7950 50  0000 C CNN
+F 1 "10K" V 5700 7950 50  0000 C CNN
+F 2 "Resistor_SMD:R_0603_1608Metric" V 5630 7950 50  0001 C CNN
+F 3 "~" H 5700 7950 50  0001 C CNN
+	1    5700 7950
+	0    1    1    0
+$EndComp
+$Comp
+L Device:R R304
+U 1 1 6292ACB5
+P 5700 8150
+F 0 "R304" V 5800 8150 50  0000 C CNN
+F 1 "47K" V 5700 8150 50  0000 C CNN
+F 2 "Resistor_SMD:R_0603_1608Metric" V 5630 8150 50  0001 C CNN
+F 3 "~" H 5700 8150 50  0001 C CNN
+	1    5700 8150
+	0    1    1    0
+$EndComp
+$Comp
+L Device:R R305
+U 1 1 62938012
+P 5700 8350
+F 0 "R305" V 5800 8350 50  0000 C CNN
+F 1 "47K" V 5700 8350 50  0000 C CNN
+F 2 "Resistor_SMD:R_0603_1608Metric" V 5630 8350 50  0001 C CNN
+F 3 "~" H 5700 8350 50  0001 C CNN
+	1    5700 8350
+	0    1    1    0
+$EndComp
+$Comp
+L Device:R R306
+U 1 1 6294520B
+P 5700 8550
+F 0 "R306" V 5800 8550 50  0000 C CNN
+F 1 "100K" V 5700 8550 50  0000 C CNN
+F 2 "Resistor_SMD:R_0603_1608Metric" V 5630 8550 50  0001 C CNN
+F 3 "~" H 5700 8550 50  0001 C CNN
+	1    5700 8550
+	0    1    1    0
+$EndComp
+$Comp
+L Device:R R307
+U 1 1 6295247C
+P 5700 8750
+F 0 "R307" V 5800 8750 50  0000 C CNN
+F 1 "100K" V 5700 8750 50  0000 C CNN
+F 2 "Resistor_SMD:R_0603_1608Metric" V 5630 8750 50  0001 C CNN
+F 3 "~" H 5700 8750 50  0001 C CNN
+	1    5700 8750
+	0    1    1    0
+$EndComp
+Wire Wire Line
+	5450 7750 5550 7750
+Wire Wire Line
+	5450 7950 5550 7950
+Wire Wire Line
+	5450 8150 5550 8150
+Wire Wire Line
+	5450 8350 5550 8350
+Wire Wire Line
+	5450 8550 5550 8550
+Wire Wire Line
+	5450 8750 5550 8750
+$Comp
+L power:+3.3V #PWR0317
+U 1 1 62A01CEF
+P 5950 7650
+F 0 "#PWR0317" H 5950 7500 50  0001 C CNN
+F 1 "+3.3V" H 5965 7823 50  0000 C CNN
+F 2 "" H 5950 7650 50  0001 C CNN
+F 3 "" H 5950 7650 50  0001 C CNN
+	1    5950 7650
+	1    0    0    -1
+$EndComp
+Wire Wire Line
+	5850 7750 5950 7750
+Wire Wire Line
+	5950 7750 5950 7650
+Wire Wire Line
+	5850 7950 5950 7950
+Wire Wire Line
+	5950 7950 5950 7750
+Connection ~ 5950 7750
+Wire Wire Line
+	5850 8150 5950 8150
+Wire Wire Line
+	5950 8150 5950 7950
+Connection ~ 5950 7950
+Wire Wire Line
+	5850 8350 5950 8350
+Wire Wire Line
+	5950 8350 5950 8150
+Connection ~ 5950 8150
+$Comp
+L power:GND #PWR0318
+U 1 1 62A3C5BF
+P 5950 8850
+F 0 "#PWR0318" H 5950 8600 50  0001 C CNN
+F 1 "GND" H 5955 8677 50  0000 C CNN
+F 2 "" H 5950 8850 50  0001 C CNN
+F 3 "" H 5950 8850 50  0001 C CNN
+	1    5950 8850
+	1    0    0    -1
+$EndComp
+Wire Wire Line
+	5850 8750 5950 8750
+Wire Wire Line
+	5950 8750 5950 8850
+Wire Wire Line
+	5850 8550 5950 8550
+Wire Wire Line
+	5950 8550 5950 8750
+Connection ~ 5950 8750
 $EndSCHEMATC

Commit message: REV3.1:  - fixed audio  - added spacers  - UART is routed through audio mux instead of I2C  - proper display connector alignment
Parts:
- R306: renamed from R305; value 47K -> 100K
- renumbered R304 to R302, R302 to R303, R303 to R304, R307 to R305, R306 to R307
Other:
- moved on the sheet: R302, R303, R304, R305, R306, R307
Changed lines of the file:
@@
 encoding utf-8
 Sheet 3 4
-Title ""
-Date ""
-Rev ""
+Title "rvPhone"
+Date "2021-12-23"
+Rev "3.1"
 Comp ""
 Comment1 ""
@@
 NoConn ~ 5750 9350
 NoConn ~ 5750 9450
+Text GLabel 5450 7750 0    55   BiDi ~ 0
+ESP32.HSPI.SS0
+Text GLabel 5450 7950 0    55   Input ~ 0
+iMX8.I2C3.SCL
 Text GLabel 5450 8150 0    55   BiDi ~ 0
-ESP32.HSPI.SS0
-Text GLabel 5450 7750 0    55   Input ~ 0
-iMX8.I2C3.SCL
-Text GLabel 5450 7950 0    55   BiDi ~ 0
 iMX8.I2C3.SDA
-Text GLabel 5450 8550 0    55   Input ~ 0
+Text GLabel 5450 8750 0    55   Input ~ 0
 iMX8.PWM1
-Text GLabel 5450 8750 0    55   BiDi ~ 0
+Text GLabel 5450 8350 0    55   BiDi ~ 0
 iMX8.GPIO5.IO29
-Text GLabel 5450 8350 0    55   BiDi ~ 0
+Text GLabel 5450 8550 0    55   BiDi ~ 0
 iMX8.GPIO5.IO28
 $Comp
-L Device:R R302
+L Device:R R303
 U 1 1 6291BF3B
-P 5700 7750
-F 0 "R302" V 5800 7750 50  0000 C CNN
-F 1 "10K" V 5700 7750 50  0000 C CNN
-F 2 "Resistor_SMD:R_0603_1608Metric" V 5630 7750 50  0001 C CNN
-F 3 "~" H 5700 7750 50  0001 C CNN
-	1    5700 7750
-	0    1    1    0
-$EndComp
-$Comp
-L Device:R R303
-U 1 1 6291C716
 P 5700 7950
 F 0 "R303" V 5800 7950 50  0000 C CNN
@@
 $Comp
 L Device:R R304
-U 1 1 6292ACB5
+U 1 1 6291C716
 P 5700 8150
 F 0 "R304" V 5800 8150 50  0000 C CNN
-F 1 "47K" V 5700 8150 50  0000 C CNN
+F 1 "10K" V 5700 8150 50  0000 C CNN
 F 2 "Resistor_SMD:R_0603_1608Metric" V 5630 8150 50  0001 C CNN
 F 3 "~" H 5700 8150 50  0001 C CNN
@@
 $EndComp
 $Comp
-L Device:R R305
+L Device:R R302
+U 1 1 6292ACB5
+P 5700 7750
+F 0 "R302" V 5800 7750 50  0000 C CNN
+F 1 "47K" V 5700 7750 50  0000 C CNN
+F 2 "Resistor_SMD:R_0603_1608Metric" V 5630 7750 50  0001 C CNN
+F 3 "~" H 5700 7750 50  0001 C CNN
+	1    5700 7750
+	0    1    1    0
+$EndComp
+$Comp
+L Device:R R306
 U 1 1 62938012
-P 5700 8350
-F 0 "R305" V 5800 8350 50  0000 C CNN
-F 1 "47K" V 5700 8350 50  0000 C CNN
-F 2 "Resistor_SMD:R_0603_1608Metric" V 5630 8350 50  0001 C CNN
-F 3 "~" H 5700 8350 50  0001 C CNN
-	1    5700 8350
-	0    1    1    0
-$EndComp
-$Comp
-L Device:R R306
-U 1 1 6294520B
 P 5700 8550
 F 0 "R306" V 5800 8550 50  0000 C CNN
@@
 $Comp
 L Device:R R307
-U 1 1 6295247C
+U 1 1 6294520B
 P 5700 8750
 F 0 "R307" V 5800 8750 50  0000 C CNN
@@
 	0    1    1    0
 $EndComp
+$Comp
+L Device:R R305
+U 1 1 6295247C
+P 5700 8350
+F 0 "R305" V 5800 8350 50  0000 C CNN
+F 1 "100K" V 5700 8350 50  0000 C CNN
+F 2 "Resistor_SMD:R_0603_1608Metric" V 5630 8350 50  0001 C CNN
+F 3 "~" H 5700 8350 50  0001 C CNN
+	1    5700 8350
+	0    1    1    0
+$EndComp
+Wire Wire Line
+	5450 7950 5550 7950
+Wire Wire Line
+	5450 8150 5550 8150
 Wire Wire Line
 	5450 7750 5550 7750
 Wire Wire Line
-	5450 7950 5550 7950
-Wire Wire Line
-	5450 8150 5550 8150
-Wire Wire Line
 	5450 8350 5550 8350
 Wire Wire Line
+	5450 8750 5550 8750
+Wire Wire Line
 	5450 8550 5550 8550
-Wire Wire Line
-	5450 8750 5550 8750
 $Comp
 L power:+3.3V #PWR0317
