File: hw/rvPhone/periph.sch (KiCad schematic (older format))
At the start: 60 parts, among them J202 Modem, J203 SIM_Card, J204 Motor, J205 Micro_SD_Card, J206 Camera, SW201 BOOT, U201 ESP32-WROOM, U202 SN74CBTLV3125, U203 TXB0104RGY, U204 TXB0104RGY, U205 DRV2605L, U206 SN74CBTLV3126, U207 TPS22917, U208 SN74LVC2G66, U209 TPS22917

Commit message: stereo audio out; lvds display; LSM9DS1 added
Parts:
- removed C208: 33pF, Capacitor_SMD:C_0603_1608Metric, symbol Device:C
- removed C220: 1uF, Capacitor_SMD:C_0603_1608Metric, symbol Device:C
- removed C221: 1000pF, Capacitor_SMD:C_0603_1608Metric, symbol Device:C
- removed JP201: SIM PULL, Connector_PinHeader_1.27mm:PinHeader_1x02_P1.27mm_Vertical, symbol Device:Jumper_NC_Small
- removed R203: 15K, Resistor_SMD:R_0603_1608Metric, symbol Device:R
- removed R211: 100K, Resistor_SMD:R_0603_1608Metric, symbol Device:R
- removed U201: ESP32-WROOM, footprints:ESP32-WROOM, symbol esp32:ESP32-WROOM
- removed U202: SN74CBTLV3125, Package_DFN_QFN:Texas_S-PVQFN-N14_ThermalVias, symbol sn74:SN74CBTLV3125
- removed U205: DRV2605L, Package_SO:VSSOP-10_3x3mm_P0.5mm, symbol drv2605l:DRV2605L
- removed U206: SN74CBTLV3126, Package_DFN_QFN:Texas_S-PVQFN-N14_ThermalVias, symbol sn74:SN74CBTLV3126
- removed U207, U209: TPS22917, footprints:Texas_R-PDSO-G6, symbol texas-tps:TPS22917
- removed U208: SN74LVC2G66, Package_SO:VSSOP-8_2.4x2.1mm_P0.5mm, symbol sn74:SN74LVC2G66
- added C226, C227, C229: 0.1uF, Capacitor_SMD:C_0603_1608Metric, symbol Device:C
- added C228: 0.01uF, Capacitor_SMD:C_0603_1608Metric, symbol Device:C
- added U201: ESP32-WROOM, footprints:ESP32-WROOM, symbol esp:ESP32-WROOM
- added U202: SN74CBTLV3125RGY, Package_DFN_QFN:Texas_S-PVQFN-N14_ThermalVias, symbol sn74:SN74CBTLV3125RGY
- added U205: DRV2605L, Package_SO:VSSOP-10_3x3mm_P0.5mm, symbol drv:DRV2605L
- added U206: TPS22917, footprints:TPS22917, symbol tps:TPS22917
- added U207: SN74LVC2G66DCU, Package_SO:VSSOP-8_2.4x2.1mm_P0.5mm, symbol sn74:SN74LVC2G66DCU
- added U208: SN74CBTLV3126RGY, Package_DFN_QFN:Texas_S-PVQFN-N14_ThermalVias, symbol sn74:SN74CBTLV3126RGY
- added U209: LSM9DS1, Package_LGA:LGA-24L_3x3.5mm_P0.43mm, symbol st:LSM9DS1
- J201: renamed from J202; footprint footprints:mpcie-socket -> footprints:Socket_mPCIe
- J205: footprint footprints:MicroSd -> footprints:microSD
- JP201: renamed from JP202; footprint Connector_PinHeader_1.27mm:PinHeader_1x03_P1.27mm_Vertical -> Jumper:SolderJumper-3_P1.3mm_Open_RoundedPad1.0x1.5mm
- JP202: renamed from JP203; footprint Connector_PinHeader_1.27mm:PinHeader_1x02_P1.27mm_Vertical -> Jumper:SolderJumper-2_P1.3mm_Open_RoundedPad1.0x1.5mm
- JP203: renamed from JP204; footprint Connector_PinHeader_1.27mm:PinHeader_1x02_P1.27mm_Vertical -> Jumper:SolderJumper-2_P1.3mm_Open_RoundedPad1.0x1.5mm
- JP204: renamed from JP205; footprint Connector_PinHeader_1.27mm:PinHeader_1x02_P1.27mm_Vertical -> Jumper:SolderJumper-2_P1.3mm_Open_RoundedPad1.0x1.5mm
- JP205: renamed from JP206; footprint Connector_PinHeader_1.27mm:PinHeader_1x02_P1.27mm_Vertical -> Jumper:SolderJumper-2_P1.3mm_Open_RoundedPad1.0x1.5mm
- renumbered C210 to C204, C211 to C205, C212 to C206, C213 to C207, C214 to C208, C224 to C209, C225 to C210, C226 to C211, C222 to C212, C223 to C213, C204 to C214, C205 to C215, C206 to C216, C207 to C217, C215 to C218, C216 to C219, C218 to C220, C219 to C221, C217 to C222, C209 to C223, C227 to C224, C228 to C225, J203 to J202, J204 to J203, J206 to J204, R207 to R203, R208 to R207, R210 to R208
Connections:
- net +3V3: now also C226.1, C227.1, U201.2 (3V3), U202.14 (VCC), U205.10 (VDD), U205.5 (EN), U205.6 (VDD/NC), U206.1 (VIN), U207.8 (VCC), U208.14 (VCC), U209.1 (VDDIO), U209.22 (VDD), U209.23 (VDD), U209.3 (VDDIO), U209.5 (SDO_A/G), U209.6 (SDO_M), U209.7 (CS_A/G), U209.8 (CS_M)
- net CAM.MISO: now also U208.5 (2A)
- net CAM.MOSI: now also U208.2 (1A)
- net CAM.PWR: now also U206.6 (VOUT)
- net CAM.SCK: now also U208.9 (3A)
- net CAM.SCL: now also U207.1 (1A)
- net CAM.SDA: now also U207.6 (2B)
- net ESP32.HSPI.MISO: now also U201.14 (IO12)
- net ESP32.HSPI.MOSI: now also U201.16 (IO13)
- net ESP32.HSPI.SCK: now also U201.13 (IO14)
- net ESP32.HSPI.SS0: now also U201.23 (IO15)
- net ESP32.IO27: now also U201.12 (IO27)
- net ESP32.IO36: now also U201.4 (SENSOR_VP)
- net ESP32.IO39: now also U201.5 (SENSOR_VN)
- net ESP32.PCM.CLK: now also U201.9 (IO33)
- net ESP32.PCM.DI: now also U201.6 (IO34)
- net ESP32.PCM.DO: now also U201.24 (IO2)
- net ESP32.PCM.SYNC: now also U201.26 (IO4)
- net ESP32.RXD0: now also U201.34 (RXD0)
- net ESP32.TXD0: now also U201.35 (TXD0)
- net ESP32.U2.DTR: now also U201.8 (IO32)
- net ESP32.U2.RI: now also U201.7 (IO35)
- net ESP32.U2.RXD: now also U201.28 (IO17)
- net ESP32.U2.TXD: now also U201.27 (IO16)
- net ESP32.VSPI.MISO: now also U201.31 (IO19), U202.5 (2A)
- net ESP32.VSPI.MOSI: now also U201.37 (IO23), U202.9 (3A)
- net ESP32.VSPI.SCK: now also U201.30 (IO18), U202.12 (4A)
- net ESP32.VSPI.SS0: now also U201.29 (IO5), U202.3 (1B)
- net GND: now also C226.2, C227.2, C228.2, C229.2, U201.1 (GND), U201.15 (GND), U201.38 (GND), U201.39 (EP), U202.15 (EP), U202.2 (1A), U202.7 (GND), U205.8 (GND), U206.2 (GND), U207.4 (GND), U208.11 (4B), U208.12 (4A), U208.13 (4OE), U208.15 (EP), U208.7 (GND), U209.14 (RES), U209.15 (RES), U209.16 (RES), U209.17 (RES), U209.18 (RES), U209.19 (GND), U209.20 (GND)
- net GPIO_20: now also U201.36 (IO22)
- net GPIO_22: now also U201.33 (IO21)
- net SPI1.MISO: now also U202.6 (2B), U208.6 (2B)
- net SPI1.MOSI: now also U202.8 (3B), U208.3 (1B)
- net SPI1.SCK: now also U202.11 (4B), U208.8 (3B)
- net SPI1.SS0: now also R203.2, U202.1 (/1OE), U202.10 (/3OE), U202.13 (/4OE), U202.4 (/2OE); no longer J205.2 (DAT3/CD), R209.2
- net SPI1.SS3: now also J205.2 (DAT3/CD), R209.2; no longer R203.2
- net TMUX.I2C0.SCL: now also U201.10 (IO25), U205.2 (SCL), U207.2 (1B), U209.2 (SCL/SPC)
- net TMUX.I2C0.SDA: now also U201.11 (IO26), U205.3 (SDA), U207.5 (2A), U209.4 (SDA/SDI/SDO)
- net WAKE: now also U201.25 (IO0)
- net at C203.1, R201.2, SW201.1: now also U201.3 (EN)
- net at C219.1: now also U205.1 (REG)
- net at J203.1 (Pin_1): now also U205.7 (OUT+)
- net at J203.2 (Pin_2): now also U205.9 (OUT-)
- net FT813.GPIO0 renamed BT81X.GPIO0
- net BT81X.GPIO0: now also U206.3 (ON), U207.3 (2C), U207.7 (1C), U208.1 (1OE), U208.10 (3OE), U208.4 (2OE)
- net FT813.GPIO3 renamed BT81X.GPIO3
- net BT81X.GPIO3: now also U205.4 (IN/TRIG)
- net iMX8_USB1_D_N renamed iMX8.USB1.D_N
- net iMX8_USB1_D_P renamed iMX8.USB1.D_P
- new net: C228.1, U209.21 (CAP)
- new net: C229.1, U209.24 (C1)
- no-connect marks 29 -> 33
Other:
- moved on the sheet: C201, C202, C204, C205, C206, C207, C208, C209, C210, C211, C212, C213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

Commit message: rev2 board
Parts:
- removed C221, C222: 0.1uF, Capacitor_SMD:C_0603_1608Metric, symbol Device:C
- removed C225: 470uF, Capacitor_Tantalum_SMD:CP_EIA-3528-21_Kemet-B, symbol Device:CP
- removed J204: Camera, Connector_PinHeader_2.54mm:PinHeader_1x08_P2.54mm_Vertical, symbol Connector_Generic:Conn_01x08
- removed R208: 100K, Resistor_SMD:R_0603_1608Metric, symbol Device:R
- removed U205: DRV2605L, Package_SO:VSSOP-10_3x3mm_P0.5mm, symbol drv:DRV2605L
- removed U206: TPS22917, footprints:TPS22917, symbol tps:TPS22917
- removed U207: SN74LVC2G66DCU, Package_SO:VSSOP-8_2.4x2.1mm_P0.5mm, symbol sn74:SN74LVC2G66DCU
- removed U208: SN74CBTLV3126RGY, Package_DFN_QFN:Texas_S-PVQFN-N14_ThermalVias, symbol sn74:SN74CBTLV3126RGY
- added C219: 10nF, Capacitor_SMD:C_0603_1608Metric, symbol Device:C
- added C228, C229, C230: 0.1uF, Capacitor_SMD:C_0603_1608Metric, symbol Device:C
- added J205: Prog, Connector_FFC-FPC:Hirose_FH12-12S-0.5SH_1x12-1MP_P0.50mm_Horizontal, symbol Connector_Generic:Conn_01x12
- added J206: Expansion, Connector_Molex:Molex_SlimStack_54722-0164_2x08_P0.50mm_Vertical, symbol Connector_Generic:Conn_02x08_Odd_Even
- added J207: Camera, Connector_Molex:Molex_SlimStack_54722-0164_2x08_P0.50mm_Vertical, symbol Connector_Generic:Conn_02x08_Odd_Even
- added R209: 4.7K, Resistor_SMD:R_0603_1608Metric, symbol Device:R
- added R210: 10K, Resistor_SMD:R_0603_1608Metric, symbol Device:R
- added SW202: PERST, Button_Switch_SMD:SW_SPST_PTS810, symbol Switch:SW_Push
- added U205: DRV2605LDGS, Package_SO:VSSOP-10_3x3mm_P0.5mm, symbol drv:DRV2605LDGS
- added U207: FT230XQ, Package_DFN_QFN:QFN-16-1EP_4x4mm_P0.65mm_EP2.1x2.1mm, symbol ftdi:FT230XQ
- added U208: TMUX154ERSW, footprints:UQFN-10_1.4x1.8mm_P0.4mm, symbol tmux:TMUX154ERSW
- C202: value 10uF -> 22uF; footprint Capacitor_SMD:C_0603_1608Metric -> Capacitor_SMD:C_0805_2012Metric
- C203: value 0.1uF -> 1uF
- C218: renamed from C224; footprint Capacitor_Tantalum_SMD:CP_EIA-3528-21_Kemet-B -> Capacitor_Tantalum_SMD:CP_EIA-7343-31_Kemet-D
- C220: value 1uF -> 10nF
- J203: footprint Connector_PinHeader_1.27mm:PinHeader_1x02_P1.27mm_Vertical -> footprints:SolderWirePad_1x02_SMD_1x2mm
- SW201: footprint footprints:Panasonic_EVPBB -> Button_Switch_SMD:SW_SPST_PTS810
- renumbered C218 to C221, C219 to C222, C226 to C223, C227 to C224, C228 to C225, C229 to C226, C223 to C227, J205 to J204, JP205 to JP204, JP204 to JP205, R209 to R208, U209 to U206
Connections:
- net +3V3: now also C228.1, C229.1, C230.1, J206.1 (Pin_1), J207.16 (Pin_16), U205.10 (VDD), U205.5 (EN), U205.6 (VDD/NC), U207.1 (VCCIO), U207.10 (VCC), U207.8 (3V3OUT), U207.9 (~RESET), U208.9 (VCC); no longer C220.1
- net BT81X.GPIO0: now also J207.8 (Pin_8)
- net BT81X.GPIO3: now also U205.4 (IN/TRIG)
- net GND: now also J204.9 (SHIELD), C219.2, C228.2, C229.2, C230.2, J205.3 (Pin_3), J205.9 (Pin_9), J206.12 (Pin_12), J206.3 (Pin_3), J206.6 (Pin_6), J206.9 (Pin_9), J207.10 (Pin_10), J207.12 (Pin_12), J207.14 (Pin_14), J207.15 (Pin_15), J207.7 (Pin_7), J207.9 (Pin_9), R210.2, SW202.2, U205.8 (GND), U207.13 (GND), U207.17 (GND), U207.3 (GND), U207.4 (~CTS), U208.4 (GND)
- net GPIO_23: now also J207.1 (Pin_1)
- net SPI1.MISO: now also J206.13 (Pin_13), J207.4 (Pin_4)
- net SPI1.MOSI: now also J206.11 (Pin_11), J207.6 (Pin_6)
- net SPI1.SCK: now also J206.15 (Pin_15), J207.2 (Pin_2)
- net TMUX.I2C0.SCL: now also J206.16 (Pin_16), J207.3 (Pin_3), U205.2 (SCL); no longer U201.10 (IO25)
- net TMUX.I2C0.SDA: now also J206.14 (Pin_14), J207.5 (Pin_5), U205.3 (SDA); no longer U201.11 (IO26)
- net ESP32.EN: now reaches C203.1, R201.2, SW201.1, U201.3 (EN)
- net ESP32.EN: now also C219.1
- net at C222.1: now also U205.1 (REG)
- net PERST: now reaches J201.22 (Pin_22)
- net PERST: now also C220.1, SW202.1
- net at J203.1 (Pin_1): now also U205.7 (OUT+)
- net at J203.2 (Pin_2): now also U205.9 (OUT-)
- net ESP32.IO39: no longer names the net of U201.5 (SENSOR_VN)
- net ESP32.RXD0 renamed ESP32.UART0.RXD
- net ESP32.UART0.RXD: now also J205.1 (Pin_1), U208.2 (A1)
- net ESP32.TXD0 renamed ESP32.UART0.TXD
- net ESP32.UART0.TXD: now also J205.2 (Pin_2), U208.6 (B1)
- new net +VSYS: J206.2 (Pin_2), J206.4 (Pin_4), J207.11 (Pin_11), J207.13 (Pin_13)
- new net JTAG_TCK: J205.4 (Pin_4)
- new net JTAG_TDI: J205.7 (Pin_7)
- new net JTAG_TDO: J205.5 (Pin_5)
- new net JTAG_TMS: J205.6 (Pin_6)
- new net JTAG_TRST_N: J205.8 (Pin_8)
- new net TMUX.GPIO0: J206.5 (Pin_5)
- new net TMUX.GPIO1: J206.7 (Pin_7)
- new net UART0.RXD: J205.11 (Pin_11), J206.8 (Pin_8), U208.1 (A0)
- new net UART0.TXD: J205.10 (Pin_10), J206.10 (Pin_10), U208.7 (B0)
- new net USB_CBUS0: U207.12 (CBUS0), U208.8 (/EN)
- new net USB_CBUS1: U207.11 (CBUS1), U208.10 (SEL)
- new net USB_CBUS3: R209.2, R210.1, U207.14 (CBUS3)
- new net USB_D+: U207.6 (USBDP)
- new net USB_D-: U207.7 (USBDM)
- new net USB_RXD: U207.2 (RXD), U208.5 (B)
- new net USB_TXD: U207.15 (TXD), U208.3 (A)
- new net VBUS: R209.1
- no-connect marks 33 -> 35
Other:
- moved on the sheet: C205, C206, C207, C208, C218, C221, C222, C223, C224, C225, C226, C227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

Commit message: temp commit for merge
Parts:
- removed J204: Micro_SD_Card, footprints:microSD, symbol Connector:Micro_SD_Card
- added C228: 22uF, Capacitor_SMD:C_0805_2012Metric, symbol Device:C
- added J204: Micro_SD_Card_Det, footprints:Molex_MicroSD-5027740891, symbol Connector:Micro_SD_Card_Det
- C219, C220: value 10nF -> 0.1uF
- J201: footprint footprints:Socket_mPCIe -> footprints:TE_mPCIe-1775862; symbol Connector_Generic:Conn_02x26_Odd_Even -> myConn:mPCIe
- JP201: value LEVEL EN -> SIMCom_EN
- SW201: value BOOT -> ESP32_RST
- SW202: value PERST -> MODEM_RST
- U202, U203, U204: footprint Package_DFN_QFN:Texas_S-PVQFN-N14_ThermalVias -> footprints:Texas_S-PVQFN-N14_ThermalVias
- renumbered C228 to C229, C229 to C230, C230 to C231
Connections:
- net labels added: ESP32.IO26, GPIO_0, SPI1.SS2
- net labels removed: ESP32.IO36, GPIO_23, SPI1.SS3
- wire segments 516 -> 524
- no-connect marks 35 -> 37
Other:
- moved on the sheet: C201, C202, C203, C204, C220, R201, R202, R203, SW201, SW202, U201, U202

Commit message: HW REV 3.0
Connections:
- net labels added: BQ.INT, ESP32_EN, ESP32_PCM_CLK, ESP32_PCM_DI, ESP32_PCM_DO, ESP32_PCM_SYNC, ESP32_UART2_DTR, ESP32_UART2_RI, ESP32_UART2_RXD, ESP32_UART2_TXD, ESP32_VSPI_MISO, ESP32_VSPI_MOSI, ESP32_VSPI_SCK, ESP32_VSPI_SS0, PCM_CLK, PCM_DI, PCM_DO, PCM_SYNC, Quectel_UART_DTR, Quectel_UART_RI, Quectel_UART_RXD, Quectel_UART_TXD, SIMCom_UART_DTR, SIMCom_UART_RI, SIMCom_UART_RXD, SIMCom_UART_TXD, VDDA
- net labels removed: ESP32.EN, ESP32.PCM.CLK, ESP32.PCM.DI, ESP32.PCM.DO, ESP32.PCM.SYNC, ESP32.U2.DTR, ESP32.U2.RI, ESP32.U2.RXD, ESP32.U2.TXD, ESP32.VSPI.MISO, ESP32.VSPI.MOSI, ESP32.VSPI.SCK, ESP32.VSPI.SS0, Modem.PCM.CLK, Modem.PCM.DI, Modem.PCM.DO, Modem.PCM.SYNC, Quectel.UART.DTR, Quectel.UART.RI, Quectel.UART.RXD, Quectel.UART.TXD, SIMCom.UART.DTR, SIMCom.UART.RI, SIMCom.UART.RXD, SIMCom.UART.TXD, TMUX.GPIO0, TMUX.GPIO1
- wire segments 524 -> 515
- no-connect marks 37 -> 40
Other:
- moved on the sheet: J207

Commit message: added pull-up pull-dn resistors; fixed input power;
Parts:
- removed R207: 100K, Resistor_SMD:R_0603_1608Metric, symbol Device:R
- renumbered R208 to R207, R209 to R208, R210 to R209
Connections:
- wire segments 515 -> 511
Changed lines of the file:
@@
 Wire Wire Line
 	7500 2850 7650 2850
-$Comp
-L Device:R R207
-U 1 1 5C88B596
-P 1850 7600
-F 0 "R207" V 1930 7600 50  0000 C CNN
-F 1 "100K" V 1850 7600 50  0000 C CNN
-F 2 "Resistor_SMD:R_0603_1608Metric" V 1780 7600 50  0001 C CNN
-F 3 "" H 1850 7600 50  0001 C CNN
-	1    1850 7600
-	-1   0    0    1
-$EndComp
 Connection ~ 3150 7150
 Connection ~ 3150 6950
@@
 	3150 6750 3150 6950
 Wire Wire Line
-	1750 7350 1850 7350
-Wire Wire Line
-	1850 7450 1850 7350
-Connection ~ 1850 7350
-Wire Wire Line
-	1850 7350 2000 7350
-Wire Wire Line
-	1850 7750 1850 8000
-Wire Wire Line
-	1850 8000 3150 8000
-Wire Wire Line
 	8650 2650 9800 2650
 Text Label 9800 2650 2    55   ~ 0
@@
 $EndComp
 $Comp
-L Device:R R208
+L Device:R R207
 U 1 1 5C6D9747
 P 1750 9350
-F 0 "R208" V 1830 9350 50  0000 C CNN
+F 0 "R207" V 1830 9350 50  0000 C CNN
 F 1 "47K" V 1750 9350 50  0000 C CNN
 F 2 "Resistor_SMD:R_0603_1608Metric" V 1680 9350 50  0001 C CNN
@@
 	9850 6700 10350 6700
 $Comp
-L Device:R R209
+L Device:R R208
 U 1 1 62EAF500
 P 12350 7400
-F 0 "R209" V 12450 7350 50  0000 L CNN
+F 0 "R208" V 12450 7350 50  0000 L CNN
 F 1 "4.7K" V 12350 7300 50  0000 L CNN
 F 2 "Resistor_SMD:R_0603_1608Metric" V 12280 7400 50  0001 C CNN
@@
 $EndComp
 $Comp
-L Device:R R210
+L Device:R R209
 U 1 1 62EAFF77
 P 12350 7800
-F 0 "R210" V 12450 7750 50  0000 L CNN
+F 0 "R209" V 12450 7750 50  0000 L CNN
 F 1 "10K" V 12350 7700 50  0000 L CNN
 F 2 "Resistor_SMD:R_0603_1608Metric" V 12280 7800 50  0001 C CNN
@@
 Text Label 4050 5400 2    55   ~ 0
 PCM_DI
+Wire Wire Line
+	1750 7350 2000 7350
 $EndSCHEMATC

Commit message: REV3.1:  - fixed audio  - added spacers  - UART is routed through audio mux instead of I2C  - proper display connector alignment
Parts:
- added J208, J209: Spacer, footprints:Spacer_small, symbol myConn:Spacer
- added JP201: PCM_EN, Jumper:SolderJumper-3_P1.3mm_Bridged2Bar12_RoundedPad1.0x1.5mm, symbol Device:Jumper_NC_Dual
- JP202: renamed from JP201; footprint Jumper:SolderJumper-3_P1.3mm_Open_RoundedPad1.0x1.5mm -> Jumper:SolderJumper-3_P1.3mm_Bridged2Bar12_RoundedPad1.0x1.5mm
- renumbered JP202 to JP203, JP203 to JP204, JP204 to JP205, JP205 to JP206
Connections:
- net labels added: +5V, I2C0.SCL, I2C0.SDA
- net labels removed: TMUX.I2C0.SCL, TMUX.I2C0.SDA, VDDA
- wire segments 511 -> 521
Other:
- moved on the sheet: C205, C206, C208, C221, C222, C231, J203, JP202, U208
